File: hardware/de0nano_cpu_card/sheets/backplane_connector.kicad_sch (KiCad schematic)
At the start: 0 parts

Commit message: Wire up all 7 schematic sheets with real nets
All architecture/sourcing decisions were already resolved; this wires
them into the actual schematic, generated from docs/cs1800.qsf and the
other docs/ files via a small purpose-built generator (tools/) rather
than hand-placing ~400 pins in the GUI:

- backplane_connector: DIN41617 31p + 13 pull-up resistors per the
  backplane pinout's *1/*2 notes
- level_shifters: all 6 SN74LVC8T245 (4 backplane + 2 future-expansion),
  DIR/OE strapping per the power-up-safe defaults in backplane_notes.md,
  plus the future-expansion 2x11 header that was previously only
  documented, not placed
- fpga_header: both DE0-Nano GPIO headers (JP1/JP2), every pin from
  cs1800.qsf, VCC3P3 wired as the board's +3V3 source
- power: backplane 5V feed header, bulk cap, PWR_FLAGs
- pico_w_bridge: Pico-W module, UART0/UART1 routing, 8 spare GPIO,
  RUN pull-up, VSYS back-feed Schottky diode
- rs232: MAX3232 (channel 1 only) + DB9, charge-pump caps
- frontpanel_io: 4 LEDs w/ series resistors, 3 switches + 3 buttons w/
  pull-ups

kicad-cli sch erc on the full hierarchy: 0 errors, 3 known/benign
warnings (custom DIN41617 footprint not drawn yet; 2 cosmetic
lib_symbol_mismatch notices on the extends-based symbols). pcb drc on
the still-placeholder board outline: 0 violations.

Co-Authored-By: Claude Sonnet 5 <noreply@anthropic.com>
Parts:
- added C3: 100pF, Capacitor_SMD:C_0603_1608Metric, symbol Device:C
- added J1: DIN41617_31P, cs1800:DIN41617_31P_Male_Angled, symbol Connector_Generic:Conn_01x31
- added R10, R12, R14, R16, R18, R2, R20, R22, R24, R26, R28, R3, R8: 10k, Resistor_SMD:R_0603_1608Metric, symbol Device:R
Connections:
- new net +5V: J1.1 (Pin_1), R10.1, R12.1, R14.1, R16.1, R18.1, R2.1, R20.1, R22.1, R24.1, R26.1, R28.1, R3.1, R8.1
- new net BP_ADDR[0]: J1.23 (Pin_23)
- new net BP_ADDR[1]: J1.21 (Pin_21)
- new net BP_ADDR[2]: J1.19 (Pin_19)
- new net BP_ADDR[3]: J1.17 (Pin_17)
- new net BP_ADDR[4]: J1.15 (Pin_15)
- new net BP_ADDR[5]: J1.13 (Pin_13)
- new net BP_ADDR[6]: J1.11 (Pin_11)
- new net BP_ADDR[7]: J1.9 (Pin_9)
- new net BP_DATA[0]: J1.22 (Pin_22), R22.2
- new net BP_DATA[1]: J1.20 (Pin_20), R20.2
- new net BP_DATA[2]: J1.18 (Pin_18), R18.2
- new net BP_DATA[3]: J1.16 (Pin_16), R16.2
- new net BP_DATA[4]: J1.14 (Pin_14), R14.2
- new net BP_DATA[5]: J1.12 (Pin_12), R12.2
- new net BP_DATA[6]: J1.10 (Pin_10), R10.2
- new net BP_DATA[7]: J1.8 (Pin_8), R8.2
- new net BP_LC: J1.2 (Pin_2), R2.2
- new net BP_N[0]: J1.29 (Pin_29)
- new net BP_N[1]: J1.27 (Pin_27)
- new net BP_N[2]: J1.25 (Pin_25)
- new net BP_Q: J1.30 (Pin_30)
- new net BP_TPA: J1.5 (Pin_5)
- new net BP_TPB: J1.7 (Pin_7)
- new net BP_nEF[0]: J1.24 (Pin_24), R24.2
- new net BP_nEF[1]: J1.26 (Pin_26), R26.2
- new net BP_nEF[2]: J1.28 (Pin_28), R28.2
- new net BP_nINT: C3.1, J1.3 (Pin_3), R3.2
- new net BP_nMRD: J1.6 (Pin_6)
- new net BP_nMWR: J1.4 (Pin_4)
- new net GND: C3.2, J1.31 (Pin_31)
