File: hardware/de0nano_cpu_card/sheets/backplane_connector.kicad_sch (KiCad schematic)
At the start: 15 parts, among them J1 DIN41617_31P

Commit message: Restore PWR_FLAGs, document 8-level-shifter GND-tie change
Schematic (user, GUI): re-added the 3 PWR_FLAG symbols (backplane +5V,
front-panel GND, Pico-W VSYS) that were deleted by mistake, clearing the
3 power_pin_not_driven ERC errors from the last round of edits. sch erc:
0 errors.

Docs: updated design_notes.md to match the user's own architecture
change made during final placement/routing -- level shifters increased
from 6 to 8 (U8/U9 added, both backplane-facing: 6 backplane + 2
future-expansion chips now), and all spare/unused channels across every
chip are now hard-tied to GND (no pull-up resistors), since DIR is
statically strapped on each chip (no bus-contention risk) and the
datasheet recommends tying off unused inputs. Updated BOM counts
accordingly (8x SN74LVC8T245, 16x decoupling caps, 25x pull-ups).
Status section and Next Steps rewritten to reflect that placement,
routing, and ground planes/via-stitching are done -- current phase is
Gerber export and JLCPCB handover.

Co-Authored-By: Claude Sonnet 5 <noreply@anthropic.com>
Changed lines of the file:
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@@
 		(company "CS1800 Project")
 	)
+	(junction
+		(at 120.65 184.15)
+		(diameter 0)
+		(color 0 0 0 0)
+	)
 	(wire
 		(pts
@@
 		(pts
 			(xy 123.19 260.35) (xy 120.65 260.35)
+		)
+		(stroke
+			(width 0)
+			(type default)
+		)
+	)
+	(wire
+		(pts
+			(xy 110.49 184.15) (xy 120.65 184.15)
 		)
 		(stroke
@@
 					(unit 1)
 				)
+			)
+		)
+	)
+	(symbol
+		(lib_id "power:PWR_FLAG")
+		(at 110.49 184.15 0)
+		(unit 1)
+		(body_style 1)
+		(exclude_from_sim no)
+		(in_bom yes)
+		(on_board yes)
+		(in_pos_files yes)
+		(dnp no)
+		(fields_autoplaced yes)
+		(property "Reference" "#FLG01"
+			(at 110.49 182.245 0)
+			(hide yes)
+			(show_name no)
+			(do_not_autoplace no)
+			(effects
+				(font
+					(size 1.27 1.27)
+				)
+			)
+		)
+		(property "Value" "PWR_FLAG"
+			(at 110.49 179.07 0)
+			(show_name no)
+			(do_not_autoplace no)
+			(effects
+				(font
+					(size 1.27 1.27)
+				)
+			)
+		)
+		(property "Footprint" ""
+			(at 110.49 184.15 0)
+			(hide yes)
+			(show_name no)
+			(do_not_autoplace no)
+			(effects
+				(font
+					(size 1.27 1.27)
+				)
+			)
+		)
+		(property "Datasheet" ""
+			(at 110.49 184.15 0)
+			(hide yes)
+			(show_name no)
+			(do_not_autoplace no)
+			(effects
+				(font
+					(size 1.27 1.27)
+				)
+			)
+		)
+		(property "Description" "Special symbol for telling ERC where power comes from"
+			(at 110.49 184.15 0)
+			(hide yes)
+			(show_name no)
+			(do_not_autoplace no)
+			(effects
+				(font
+					(size 1.27 1.27)
+				)
+			)
+		)
+		(pin "1"
+		)
+		(instances
+			(project "de0nano_cpu_card"
+				(path "/0daab69e-2257-45dd-abd7-efbe947cce3e/4f6bbb95-6697-43c0-83d6-5afb3916ffb4"
+					(reference "#FLG01")
+					(unit 1)
+				)
