File: hardware/de0nano_cpu_card/sheets/fpga_header.kicad_sch (KiCad schematic)
At the start: 0 parts

Commit message: Wire up all 7 schematic sheets with real nets
All architecture/sourcing decisions were already resolved; this wires
them into the actual schematic, generated from docs/cs1800.qsf and the
other docs/ files via a small purpose-built generator (tools/) rather
than hand-placing ~400 pins in the GUI:

- backplane_connector: DIN41617 31p + 13 pull-up resistors per the
  backplane pinout's *1/*2 notes
- level_shifters: all 6 SN74LVC8T245 (4 backplane + 2 future-expansion),
  DIR/OE strapping per the power-up-safe defaults in backplane_notes.md,
  plus the future-expansion 2x11 header that was previously only
  documented, not placed
- fpga_header: both DE0-Nano GPIO headers (JP1/JP2), every pin from
  cs1800.qsf, VCC3P3 wired as the board's +3V3 source
- power: backplane 5V feed header, bulk cap, PWR_FLAGs
- pico_w_bridge: Pico-W module, UART0/UART1 routing, 8 spare GPIO,
  RUN pull-up, VSYS back-feed Schottky diode
- rs232: MAX3232 (channel 1 only) + DB9, charge-pump caps
- frontpanel_io: 4 LEDs w/ series resistors, 3 switches + 3 buttons w/
  pull-ups

kicad-cli sch erc on the full hierarchy: 0 errors, 3 known/benign
warnings (custom DIN41617 footprint not drawn yet; 2 cosmetic
lib_symbol_mismatch notices on the extends-based symbols). pcb drc on
the still-placeholder board outline: 0 violations.

Co-Authored-By: Claude Sonnet 5 <noreply@anthropic.com>
Parts:
- added J1: GPIO_0_JP1, Connector_IDC:IDC-Header_2x20_P2.54mm_Vertical, symbol Connector_Generic:Conn_02x20_Odd_Even
- added J2: GPIO_1_JP2, Connector_IDC:IDC-Header_2x20_P2.54mm_Vertical, symbol Connector_Generic:Conn_02x20_Odd_Even
Connections:
- new net +3V3: J1.29 (Pin_29)
- new net ADDR[0]: J1.31 (Pin_31)
- new net ADDR[1]: J1.28 (Pin_28)
- new net ADDR[2]: J1.27 (Pin_27)
- new net ADDR[3]: J1.26 (Pin_26)
- new net ADDR[4]: J1.25 (Pin_25)
- new net ADDR[5]: J1.24 (Pin_24)
- new net ADDR[6]: J1.23 (Pin_23)
- new net ADDR[7]: J1.22 (Pin_22)
- new net BUF_nOE: J1.13 (Pin_13)
- new net BUT_qef4: J2.40 (Pin_40)
- new net BUT_reset: J2.39 (Pin_39)
- new net BUT_step: J2.38 (Pin_38)
- new net CS[0]: J2.18 (Pin_18)
- new net CS[1]: J2.19 (Pin_19)
- new net DATA[0]: J1.21 (Pin_21)
- new net DATA[1]: J1.20 (Pin_20)
- new net DATA[2]: J1.19 (Pin_19)
- new net DATA[3]: J1.18 (Pin_18)
- new net DATA[4]: J1.17 (Pin_17)
- new net DATA[5]: J1.16 (Pin_16)
- new net DATA[6]: J1.15 (Pin_15)
- new net DATA[7]: J1.14 (Pin_14)
- new net DATA_DIR: J1.9 (Pin_9)
- new net DATA_nOE: J1.10 (Pin_10)
- new net EX_IN[0]: J2.22 (Pin_22)
- new net EX_IN[1]: J2.23 (Pin_23)
- new net EX_OUT[0]: J2.20 (Pin_20)
- new net EX_OUT[1]: J2.21 (Pin_21)
- new net GND: J1.12 (Pin_12), J1.30 (Pin_30), J2.12 (Pin_12), J2.30 (Pin_30)
- new net LC: J1.2 (Pin_2)
- new net LED1_fetch: J2.31 (Pin_31)
- new net LED2_execute: J2.32 (Pin_32)
- new net LED3_interrupt: J2.33 (Pin_33)
- new net LED4_Q: J2.34 (Pin_34)
- new net N[0]: J1.37 (Pin_37)
- new net N[1]: J1.36 (Pin_36)
- new net N[2]: J1.35 (Pin_35)
- new net PICO[0]: J2.17 (Pin_17)
- new net PICO[1]: J2.16 (Pin_16)
- new net PICO[2]: J2.15 (Pin_15)
- new net PICO[3]: J2.14 (Pin_14)
- new net PICO[4]: J2.13 (Pin_13)
- new net PICO[5]: J2.10 (Pin_10)
- new net PICO[6]: J2.9 (Pin_9)
- new net PICO[7]: J2.8 (Pin_8)
- new net Q: J1.38 (Pin_38)
- new net SW_LC_off: J2.37 (Pin_37)
- new net SW_dog: J2.36 (Pin_36)
- new net SW_halt: J2.35 (Pin_35)
- new net TPA: J1.6 (Pin_6)
- new net TPB: J1.8 (Pin_8)
- new net UART0_RXD: J2.4 (Pin_4)
- new net UART0_TXD: J2.2 (Pin_2)
- new net nCLEAR: J2.25 (Pin_25)
- new net nDMA_IN: J2.28 (Pin_28)
- new net nDMA_OUT: J2.27 (Pin_27)
- new net nEF[0]: J1.32 (Pin_32)
- new net nEF[1]: J1.33 (Pin_33)
- new net nEF[2]: J1.34 (Pin_34)
- new net nEF[3]: J2.24 (Pin_24)
- new net nINT: J1.4 (Pin_4)
- new net nMRD: J1.7 (Pin_7)
- new net nMWR: J1.5 (Pin_5)
- new net nWAIT: J2.26 (Pin_26)
- no-connect marks 0 -> 12
