File: hardware/de0nano_cpu_card/sheets/fpga_header.kicad_sch (KiCad schematic)
At the start: 6 parts, among them J1 GPIO_0_JP1, J2 GPIO_1_JP2

Commit message: Fix cross-sheet reference-designator collisions (required for PCB work)
Each build_*.py numbered its own parts independently (R1, C1, J1, U1,
etc. each starting fresh per sheet), which kicad-cli sch erc never
flagged -- ERC resolves connectivity by net name, not reference, so
duplicate refs across sheets are invisible to it. Only surfaced when
starting PCB work: `kicad-cli sch export netlist` warned about
annotation errors, and its (components) section showed 19 reference
names each silently mapping to 2-4 different real parts (89 components
total, e.g. "R1" meant three unrelated resistors on three sheets).

Fixed via tools/patch_reannotate_global.py: 60 references renumbered
to be globally unique, processed in root-sheet hierarchy order.
Required updating BOTH the visible (property "Reference" ...) field
and the (reference ...) inside each symbol's (instances ...) block --
the netlist exporter reads only the latter, so a first attempt that
touched just the property field silently had no effect on the
netlist. Both quirks documented in tools/README.md.

Verified: netlist's (components) section now has zero duplicate refs
(89 unique). sch erc: still 0 errors. pcb drc: still 0 violations.

Co-Authored-By: Claude Sonnet 5 <noreply@anthropic.com>
Parts:
- renumbered J1 to J3, J2 to J4, R20 to R28, R21 to R29, R22 to R30, R23 to R31
Changed lines of the file:
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@@
 		(in_pos_files yes)
 		(dnp no)
-		(property "Reference" "J2"
+		(property "Reference" "J4"
 			(at 219.71 43.53 0)
 			(show_name no)
@@
 			(project "de0nano_cpu_card"
 				(path "/0daab69e-2257-45dd-abd7-efbe947cce3e/a56ed679-b35c-49f9-890d-ca9b02a60560"
-					(reference "J2")
+					(reference "J4")
 					(unit 1)
 				)
@@
 		(in_pos_files yes)
 		(dnp no)
-		(property "Reference" "R23"
+		(property "Reference" "R31"
 			(at 316.23 80.36 0)
 			(show_name no)
@@
 			(project "de0nano_cpu_card"
 				(path "/0daab69e-2257-45dd-abd7-efbe947cce3e/a56ed679-b35c-49f9-890d-ca9b02a60560"
-					(reference "R23")
+					(reference "R31")
 					(unit 1)
 				)
@@
 		(in_pos_files yes)
 		(dnp no)
-		(property "Reference" "R22"
+		(property "Reference" "R30"
 			(at 316.23 65.12 0)
 			(show_name no)
@@
 			(project "de0nano_cpu_card"
 				(path "/0daab69e-2257-45dd-abd7-efbe947cce3e/a56ed679-b35c-49f9-890d-ca9b02a60560"
-					(reference "R22")
+					(reference "R30")
 					(unit 1)
 				)
@@
 		(in_pos_files yes)
 		(dnp no)
-		(property "Reference" "J1"
+		(property "Reference" "J3"
 			(at 49.53 43.53 0)
 			(show_name no)
@@
 			(project "de0nano_cpu_card"
 				(path "/0daab69e-2257-45dd-abd7-efbe947cce3e/a56ed679-b35c-49f9-890d-ca9b02a60560"
-					(reference "J1")
+					(reference "J3")
 					(unit 1)
 				)
@@
 		(in_pos_files yes)
 		(dnp no)
-		(property "Reference" "R20"
+		(property "Reference" "R28"
 			(at 316.23 35.91 0)
 			(show_name no)
@@
 			(project "de0nano_cpu_card"
 				(path "/0daab69e-2257-45dd-abd7-efbe947cce3e/a56ed679-b35c-49f9-890d-ca9b02a60560"
-					(reference "R20")
+					(reference "R28")
 					(unit 1)
 				)
@@
 		(in_pos_files yes)
 		(dnp no)
-		(property "Reference" "R21"
+		(property "Reference" "R29"
 			(at 316.23 51.15 0)
 			(show_name no)
@@
 			(project "de0nano_cpu_card"
 				(path "/0daab69e-2257-45dd-abd7-efbe947cce3e/a56ed679-b35c-49f9-890d-ca9b02a60560"
-					(reference "R21")
+					(reference "R29")
 					(unit 1)
 				)
