File: hardware/de0nano_cpu_card/sheets/frontpanel_io.kicad_sch (KiCad schematic)
At the start: 0 parts

Commit message: Wire up all 7 schematic sheets with real nets
All architecture/sourcing decisions were already resolved; this wires
them into the actual schematic, generated from docs/cs1800.qsf and the
other docs/ files via a small purpose-built generator (tools/) rather
than hand-placing ~400 pins in the GUI:

- backplane_connector: DIN41617 31p + 13 pull-up resistors per the
  backplane pinout's *1/*2 notes
- level_shifters: all 6 SN74LVC8T245 (4 backplane + 2 future-expansion),
  DIR/OE strapping per the power-up-safe defaults in backplane_notes.md,
  plus the future-expansion 2x11 header that was previously only
  documented, not placed
- fpga_header: both DE0-Nano GPIO headers (JP1/JP2), every pin from
  cs1800.qsf, VCC3P3 wired as the board's +3V3 source
- power: backplane 5V feed header, bulk cap, PWR_FLAGs
- pico_w_bridge: Pico-W module, UART0/UART1 routing, 8 spare GPIO,
  RUN pull-up, VSYS back-feed Schottky diode
- rs232: MAX3232 (channel 1 only) + DB9, charge-pump caps
- frontpanel_io: 4 LEDs w/ series resistors, 3 switches + 3 buttons w/
  pull-ups

kicad-cli sch erc on the full hierarchy: 0 errors, 3 known/benign
warnings (custom DIN41617 footprint not drawn yet; 2 cosmetic
lib_symbol_mismatch notices on the extends-based symbols). pcb drc on
the still-placeholder board outline: 0 violations.

Co-Authored-By: Claude Sonnet 5 <noreply@anthropic.com>
Parts:
- added D1: LED_Green, LED_THT:LED_D3.0mm, symbol Device:LED
- added D2: LED_Yellow, LED_THT:LED_D3.0mm, symbol Device:LED
- added D3, D4: LED_Red, LED_THT:LED_D3.0mm, symbol Device:LED
- added R_D1, R_D2, R_D3, R_D4: 220, Resistor_SMD:R_0603_1608Metric, symbol Device:R
- added R_SW1, R_SW2, R_SW3, R_SW4, R_SW5, R_SW6: 10k, Resistor_SMD:R_0603_1608Metric, symbol Device:R
- added SW1: Rocker_run/halt, Connector_PinHeader_2.54mm:PinHeader_1x02_P2.54mm_Vertical, symbol Connector_Generic:Conn_01x02
- added SW2: Rocker_dog_off, Connector_PinHeader_2.54mm:PinHeader_1x02_P2.54mm_Vertical, symbol Connector_Generic:Conn_01x02
- added SW3: Rocker_LC_off, Connector_PinHeader_2.54mm:PinHeader_1x02_P2.54mm_Vertical, symbol Connector_Generic:Conn_01x02
- added SW4: Button_step, Connector_PinHeader_2.54mm:PinHeader_1x02_P2.54mm_Vertical, symbol Connector_Generic:Conn_01x02
- added SW5: Button_reset, Connector_PinHeader_2.54mm:PinHeader_1x02_P2.54mm_Vertical, symbol Connector_Generic:Conn_01x02
- added SW6: Button_qef4, Connector_PinHeader_2.54mm:PinHeader_1x02_P2.54mm_Vertical, symbol Connector_Generic:Conn_01x02
Connections:
- new net +3V3: R_SW1.2, R_SW2.2, R_SW3.2, R_SW4.2, R_SW5.2, R_SW6.2
- new net BUT_qef4: R_SW6.1, SW6.1 (Pin_1)
- new net BUT_reset: R_SW5.1, SW5.1 (Pin_1)
- new net BUT_step: R_SW4.1, SW4.1 (Pin_1)
- new net GND: D1.1 (K), D2.1 (K), D3.1 (K), D4.1 (K), SW1.2 (Pin_2), SW2.2 (Pin_2), SW3.2 (Pin_2), SW4.2 (Pin_2), SW5.2 (Pin_2), SW6.2 (Pin_2)
- new net LED1_fetch: R_D1.1
- new net LED1_fetch_A: D1.2 (A), R_D1.2
- new net LED2_execute: R_D2.1
- new net LED2_execute_A: D2.2 (A), R_D2.2
- new net LED3_interrupt: R_D3.1
- new net LED3_interrupt_A: D3.2 (A), R_D3.2
- new net LED4_Q: R_D4.1
- new net LED4_Q_A: D4.2 (A), R_D4.2
- new net SW_LC_off: R_SW3.1, SW3.1 (Pin_1)
- new net SW_dog: R_SW2.1, SW2.1 (Pin_1)
- new net SW_halt: R_SW1.1, SW1.1 (Pin_1)
