File: hardware/de0nano_cpu_card/sheets/frontpanel_io.kicad_sch (KiCad schematic)
At the start: 20 parts, among them SW1 Rocker_run/halt, SW2 Rocker_dog_off, SW3 Rocker_LC_off, SW4 Button_step, SW5 Button_reset, SW6 Button_qef4

Commit message: Fix cross-sheet reference-designator collisions (required for PCB work)
Each build_*.py numbered its own parts independently (R1, C1, J1, U1,
etc. each starting fresh per sheet), which kicad-cli sch erc never
flagged -- ERC resolves connectivity by net name, not reference, so
duplicate refs across sheets are invisible to it. Only surfaced when
starting PCB work: `kicad-cli sch export netlist` warned about
annotation errors, and its (components) section showed 19 reference
names each silently mapping to 2-4 different real parts (89 components
total, e.g. "R1" meant three unrelated resistors on three sheets).

Fixed via tools/patch_reannotate_global.py: 60 references renumbered
to be globally unique, processed in root-sheet hierarchy order.
Required updating BOTH the visible (property "Reference" ...) field
and the (reference ...) inside each symbol's (instances ...) block --
the netlist exporter reads only the latter, so a first attempt that
touched just the property field silently had no effect on the
netlist. Both quirks documented in tools/README.md.

Verified: netlist's (components) section now has zero duplicate refs
(89 unique). sch erc: still 0 errors. pcb drc: still 0 violations.

Co-Authored-By: Claude Sonnet 5 <noreply@anthropic.com>
Parts:
- renumbered D1 to D2, D2 to D3, D3 to D4, D4 to D5
Changed lines of the file:
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@@
 		(in_pos_files yes)
 		(dnp no)
-		(property "Reference" "D1"
+		(property "Reference" "D2"
 			(at 30.48 24.48 0)
 			(show_name no)
@@
 			(project "de0nano_cpu_card"
 				(path "/0daab69e-2257-45dd-abd7-efbe947cce3e/5bdfddb1-6b11-40ff-a5b3-24c3d0c519a0"
-					(reference "D1")
+					(reference "D2")
 					(unit 1)
 				)
@@
 		(in_pos_files yes)
 		(dnp no)
-		(property "Reference" "D2"
+		(property "Reference" "D3"
 			(at 59.69 24.48 0)
 			(show_name no)
@@
 			(project "de0nano_cpu_card"
 				(path "/0daab69e-2257-45dd-abd7-efbe947cce3e/5bdfddb1-6b11-40ff-a5b3-24c3d0c519a0"
-					(reference "D2")
+					(reference "D3")
 					(unit 1)
 				)
@@
 		(in_pos_files yes)
 		(dnp no)
-		(property "Reference" "D4"
+		(property "Reference" "D5"
 			(at 119.38 24.48 0)
 			(show_name no)
@@
 			(project "de0nano_cpu_card"
 				(path "/0daab69e-2257-45dd-abd7-efbe947cce3e/5bdfddb1-6b11-40ff-a5b3-24c3d0c519a0"
-					(reference "D4")
+					(reference "D5")
 					(unit 1)
 				)
@@
 		(in_pos_files yes)
 		(dnp no)
-		(property "Reference" "D3"
+		(property "Reference" "D4"
 			(at 90.17 24.48 0)
 			(show_name no)
@@
 			(project "de0nano_cpu_card"
 				(path "/0daab69e-2257-45dd-abd7-efbe947cce3e/5bdfddb1-6b11-40ff-a5b3-24c3d0c519a0"
-					(reference "D3")
-					(unit 1)
-				)
+					(reference "D4")
+					(unit 1)
+				)
