File: hardware/de0nano_cpu_card/sheets/frontpanel_io.kicad_sch (KiCad schematic)
At the start: 20 parts, among them SW1 Rocker_run/halt, SW2 Rocker_dog_off, SW3 Rocker_LC_off, SW4 Button_step, SW5 Button_reset, SW6 Button_qef4

Commit message: Restore PWR_FLAGs, document 8-level-shifter GND-tie change
Schematic (user, GUI): re-added the 3 PWR_FLAG symbols (backplane +5V,
front-panel GND, Pico-W VSYS) that were deleted by mistake, clearing the
3 power_pin_not_driven ERC errors from the last round of edits. sch erc:
0 errors.

Docs: updated design_notes.md to match the user's own architecture
change made during final placement/routing -- level shifters increased
from 6 to 8 (U8/U9 added, both backplane-facing: 6 backplane + 2
future-expansion chips now), and all spare/unused channels across every
chip are now hard-tied to GND (no pull-up resistors), since DIR is
statically strapped on each chip (no bus-contention risk) and the
datasheet recommends tying off unused inputs. Updated BOM counts
accordingly (8x SN74LVC8T245, 16x decoupling caps, 25x pull-ups).
Status section and Next Steps rewritten to reflect that placement,
routing, and ground planes/via-stitching are done -- current phase is
Gerber export and JLCPCB handover.

Co-Authored-By: Claude Sonnet 5 <noreply@anthropic.com>
Changed lines of the file:
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@@
 		(company "CS1800 Project")
 	)
+	(junction
+		(at 186.69 149.86)
+		(diameter 0)
+		(color 0 0 0 0)
+	)
 	(wire
 		(pts
@@
 	(wire
 		(pts
-			(xy 115.57 30.48) (xy 113.03 30.48)
-		)
-		(stroke
-			(width 0)
-			(type default)
-		)
-	)
-	(wire
-		(pts
 			(xy 34.29 149.86) (xy 36.83 149.86)
 		)
@@
 	(wire
 		(pts
+			(xy 186.69 149.86) (xy 193.04 149.86)
+		)
+		(stroke
+			(width 0)
+			(type default)
+		)
+	)
+	(wire
+		(pts
 			(xy 53.34 59.69) (xy 55.88 59.69)
 		)
@@
 	(wire
 		(pts
+			(xy 106.68 30.48) (xy 115.57 30.48)
+		)
+		(stroke
+			(width 0)
+			(type default)
+		)
+	)
+	(wire
+		(pts
 			(xy 144.78 137.16) (xy 144.78 149.86)
 		)
@@
 	)
 	(symbol
+		(lib_id "power:PWR_FLAG")
+		(at 193.04 149.86 0)
+		(unit 1)
+		(body_style 1)
+		(exclude_from_sim no)
+		(in_bom yes)
+		(on_board yes)
+		(in_pos_files yes)
+		(dnp no)
+		(fields_autoplaced yes)
+		(property "Reference" "#FLG04"
+			(at 193.04 147.955 0)
+			(hide yes)
+			(show_name no)
+			(do_not_autoplace no)
+			(effects
+				(font
+					(size 1.27 1.27)
+				)
+			)
+		)
+		(property "Value" "PWR_FLAG"
+			(at 193.04 144.78 0)
+			(show_name no)
+			(do_not_autoplace no)
+			(effects
+				(font
+					(size 1.27 1.27)
+				)
+			)
+		)
+		(property "Footprint" ""
+			(at 193.04 149.86 0)
+			(hide yes)
+			(show_name no)
+			(do_not_autoplace no)
+			(effects
+				(font
+					(size 1.27 1.27)
+				)
+			)
+		)
+		(property "Datasheet" ""
+			(at 193.04 149.86 0)
+			(hide yes)
+			(show_name no)
+			(do_not_autoplace no)
+			(effects
+				(font
+					(size 1.27 1.27)
+				)
+			)
+		)
+		(property "Description" "Special symbol for telling ERC where power comes from"
+			(at 193.04 149.86 0)
+			(hide yes)
+			(show_name no)
+			(do_not_autoplace no)
+			(effects
+				(font
+					(size 1.27 1.27)
+				)
+			)
+		)
+		(pin "1"
+		)
+		(instances
+			(project "de0nano_cpu_card"
+				(path "/0daab69e-2257-45dd-abd7-efbe947cce3e/5bdfddb1-6b11-40ff-a5b3-24c3d0c519a0"
+					(reference "#FLG04")
+					(unit 1)
+				)
+			)
+		)
+	)
+	(symbol
 		(lib_id "Device:R")
 		(at 90.17 149.86 90)
@@
 	(symbol
 		(lib_id "power:GND")
-		(at 113.03 30.48 0)
+		(at 106.68 30.48 0)
 		(unit 1)
 		(body_style 1)
@@
 		(dnp no)
 		(property "Reference" "#PWR034"
-			(at 113.03 30.48 0)
+			(at 106.68 30.48 0)
 			(hide yes)
 			(show_name no)
@@
 		)
 		(property "Value" "GND"
-			(at 113.03 27.94 0)
+			(at 106.68 27.94 0)
 			(show_name no)
 			(do_not_autoplace no)
@@
 		)
 		(property "Footprint" ""
-			(at 113.03 30.48 0)
+			(at 106.68 30.48 0)
 			(show_name no)
 			(do_not_autoplace no)
@@
 		)
 		(property "Datasheet" ""
-			(at 113.03 30.48 0)
+			(at 106.68 30.48 0)
 			(show_name no)
 			(do_not_autoplace no)
@@
 		)
 		(property "Description" ""
-			(at 113.03 30.48 0)
+			(at 106.68 30.48 0)
 			(show_name no)
 			(do_not_autoplace no)
