File: hardware/de0nano_cpu_card/sheets/level_shifters.kicad_sch (KiCad schematic)
At the start: 0 parts

Commit message: Wire up all 7 schematic sheets with real nets
All architecture/sourcing decisions were already resolved; this wires
them into the actual schematic, generated from docs/cs1800.qsf and the
other docs/ files via a small purpose-built generator (tools/) rather
than hand-placing ~400 pins in the GUI:

- backplane_connector: DIN41617 31p + 13 pull-up resistors per the
  backplane pinout's *1/*2 notes
- level_shifters: all 6 SN74LVC8T245 (4 backplane + 2 future-expansion),
  DIR/OE strapping per the power-up-safe defaults in backplane_notes.md,
  plus the future-expansion 2x11 header that was previously only
  documented, not placed
- fpga_header: both DE0-Nano GPIO headers (JP1/JP2), every pin from
  cs1800.qsf, VCC3P3 wired as the board's +3V3 source
- power: backplane 5V feed header, bulk cap, PWR_FLAGs
- pico_w_bridge: Pico-W module, UART0/UART1 routing, 8 spare GPIO,
  RUN pull-up, VSYS back-feed Schottky diode
- rs232: MAX3232 (channel 1 only) + DB9, charge-pump caps
- frontpanel_io: 4 LEDs w/ series resistors, 3 switches + 3 buttons w/
  pull-ups

kicad-cli sch erc on the full hierarchy: 0 errors, 3 known/benign
warnings (custom DIN41617 footprint not drawn yet; 2 cosmetic
lib_symbol_mismatch notices on the extends-based symbols). pcb drc on
the still-placeholder board outline: 0 violations.

Co-Authored-By: Claude Sonnet 5 <noreply@anthropic.com>
Parts:
- added J2: EXP_HEADER_2x11, Connector_PinHeader_2.54mm:PinHeader_2x11_P2.54mm_Vertical, symbol Connector_Generic:Conn_02x11_Odd_Even
- added R1, R2, R3: 10k, Resistor_SMD:R_0603_1608Metric, symbol Device:R
- added U1, U2, U3, U4, U5, U6: SN74LVC8T245, Package_SO:TSSOP-24_4.4x7.8mm_P0.65mm, symbol Logic_LevelTranslator:SN74LVC8T245
Connections:
- new net +3V3: R2.1, R3.1, U1.1 (V_{CCA}), U1.2 (DIR), U2.1 (V_{CCA}), U2.2 (DIR), U3.1 (V_{CCA}), U4.1 (V_{CCA}), U5.1 (V_{CCA}), U5.2 (DIR), U6.1 (V_{CCA})
- new net +5V: U1.23 (V_{CCB}), U1.24 (V_{CCB}), U2.23 (V_{CCB}), U2.24 (V_{CCB}), U3.23 (V_{CCB}), U3.24 (V_{CCB}), U4.23 (V_{CCB}), U4.24 (V_{CCB}), U5.23 (V_{CCB}), U5.24 (V_{CCB}), U6.23 (V_{CCB}), U6.24 (V_{CCB})
- new net ADDR[0]: U1.10 (A8)
- new net ADDR[1]: U1.9 (A7)
- new net ADDR[2]: U1.8 (A6)
- new net ADDR[3]: U1.7 (A5)
- new net ADDR[4]: U1.6 (A4)
- new net ADDR[5]: U1.5 (A3)
- new net ADDR[6]: U1.4 (A2)
- new net ADDR[7]: U1.3 (A1)
- new net BP_ADDR[0]: U1.14 (B8)
- new net BP_ADDR[1]: U1.15 (B7)
- new net BP_ADDR[2]: U1.16 (B6)
- new net BP_ADDR[3]: U1.17 (B5)
- new net BP_ADDR[4]: U1.18 (B4)
- new net BP_ADDR[5]: U1.19 (B3)
- new net BP_ADDR[6]: U1.20 (B2)
- new net BP_ADDR[7]: U1.21 (B1)
- new net BP_DATA[0]: U3.14 (B8)
- new net BP_DATA[1]: U3.15 (B7)
- new net BP_DATA[2]: U3.16 (B6)
- new net BP_DATA[3]: U3.17 (B5)
- new net BP_DATA[4]: U3.18 (B4)
- new net BP_DATA[5]: U3.19 (B3)
- new net BP_DATA[6]: U3.20 (B2)
- new net BP_DATA[7]: U3.21 (B1)
- new net BP_LC: U4.21 (B1)
- new net BP_N[0]: U2.15 (B7)
- new net BP_N[1]: U2.16 (B6)
- new net BP_N[2]: U2.17 (B5)
- new net BP_Q: U2.14 (B8)
- new net BP_TPA: U2.20 (B2)
- new net BP_TPB: U2.18 (B4)
- new net BP_nEF[0]: U4.19 (B3)
- new net BP_nEF[1]: U4.18 (B4)
- new net BP_nEF[2]: U4.17 (B5)
- new net BP_nINT: U4.20 (B2)
- new net BP_nMRD: U2.19 (B3)
- new net BP_nMWR: U2.21 (B1)
- new net BUF_nOE: R3.2, U1.22 (~{OE}), U2.22 (~{OE})
- new net CS[0]: U5.3 (A1)
- new net CS[1]: U5.4 (A2)
- new net DATA[0]: U3.10 (A8)
- new net DATA[1]: U3.9 (A7)
- new net DATA[2]: U3.8 (A6)
- new net DATA[3]: U3.7 (A5)
- new net DATA[4]: U3.6 (A4)
- new net DATA[5]: U3.5 (A3)
- new net DATA[6]: U3.4 (A2)
- new net DATA[7]: U3.3 (A1)
- new net DATA_DIR: R1.1, U3.2 (DIR)
- new net DATA_nOE: R2.2, U3.22 (~{OE})
- new net EXP_CS[0]: J2.1 (Pin_1), U5.21 (B1)
- new net EXP_CS[1]: J2.3 (Pin_3), U5.20 (B2)
- new net EXP_EX_IN[0]: J2.9 (Pin_9), U6.21 (B1)
- new net EXP_EX_IN[1]: J2.11 (Pin_11), U6.20 (B2)
- new net EXP_EX_OUT[0]: J2.5 (Pin_5), U5.19 (B3)
- new net EXP_EX_OUT[1]: J2.7 (Pin_7), U5.18 (B4)
- new net EXP_nCLEAR: J2.15 (Pin_15), U6.18 (B4)
- new net EXP_nDMA_IN: J2.21 (Pin_21), U6.15 (B7)
- new net EXP_nDMA_OUT: J2.19 (Pin_19), U6.16 (B6)
- new net EXP_nEF[3]: J2.13 (Pin_13), U6.19 (B3)
- new net EXP_nWAIT: J2.17 (Pin_17), U6.17 (B5)
- new net EX_IN[0]: U6.3 (A1)
- new net EX_IN[1]: U6.4 (A2)
- new net EX_OUT[0]: U5.5 (A3)
- new net EX_OUT[1]: U5.6 (A4)
- new net GND: J2.10 (Pin_10), J2.12 (Pin_12), J2.14 (Pin_14), J2.16 (Pin_16), J2.18 (Pin_18), J2.2 (Pin_2), J2.20 (Pin_20), J2.22 (Pin_22), J2.4 (Pin_4), J2.6 (Pin_6), J2.8 (Pin_8), R1.2, U1.11 (GND), U1.12 (GND), U1.13 (GND), U2.11 (GND), U2.12 (GND), U2.13 (GND), U3.11 (GND), U3.12 (GND), U3.13 (GND), U4.11 (GND), U4.12 (GND), U4.13 (GND), U4.2 (DIR), U4.22 (~{OE}), U5.11 (GND), U5.12 (GND), U5.13 (GND), U5.22 (~{OE}), U6.11 (GND), U6.12 (GND), U6.13 (GND), U6.2 (DIR), U6.22 (~{OE})
- new net LC: U4.3 (A1)
- new net N[0]: U2.9 (A7)
- new net N[1]: U2.8 (A6)
- new net N[2]: U2.7 (A5)
- new net Q: U2.10 (A8)
- new net TPA: U2.4 (A2)
- new net TPB: U2.6 (A4)
- new net nCLEAR: U6.6 (A4)
- new net nDMA_IN: U6.9 (A7)
- new net nDMA_OUT: U6.8 (A6)
- new net nEF[0]: U4.5 (A3)
- new net nEF[1]: U4.6 (A4)
- new net nEF[2]: U4.7 (A5)
- new net nEF[3]: U6.5 (A3)
- new net nINT: U4.4 (A2)
- new net nMRD: U2.5 (A3)
- new net nMWR: U2.3 (A1)
- new net nWAIT: U6.7 (A5)
- no-connect marks 0 -> 16
Other:
- title: Level Shifters (4x SN74LVC8T245) -> Level Shifters (6x SN74LVC8T245)
