File: hardware/de0nano_cpu_card/sheets/level_shifters.kicad_sch (KiCad schematic)
At the start: 21 parts, among them J2 EXP_HEADER_2x11, U1 SN74LVC8T245, U2 SN74LVC8T245, U3 SN74LVC8T245, U4 SN74LVC8T245, U5 SN74LVC8T245, U6 SN74LVC8T245

Commit message: Add decoupling caps for all 6 level shifters (12x 100nF)
Each SN74LVC8T245 needs a 100nF ceramic cap on both supplies (VCCA=3V3,
VCCB=5V) -- 12 caps total (C1-C12), added via a surgical patch script
(tools/patch_level_shifters_decoupling.py) to preserve the user's GUI
layout, same approach as the previous pull-up/series-resistor patches.

Noted in design_notes.md as a PCB-layout requirement, not just a
schematic one: each cap needs to sit physically close to its IC's
VCCA/VCCB pin when placing parts, which the schematic placement alone
doesn't guarantee.

sch erc: still 0 errors, same warnings as before. pcb drc: 0 violations.

Co-Authored-By: Claude Sonnet 5 <noreply@anthropic.com>
Parts:
- added C1, C10, C11, C12, C2, C3, C4, C5, C6, C7, C8, C9: 100nF, Capacitor_SMD:C_0603_1608Metric, symbol Device:C
Connections:
- net +3V3: now also C1.1, C11.1, C3.1, C5.1, C7.1, C9.1
- net +5V: now also C10.1, C12.1, C2.1, C4.1, C6.1, C8.1
- net GND: now also C1.2, C10.2, C11.2, C12.2, C2.2, C3.2, C4.2, C5.2, C6.2, C7.2, C8.2, C9.2
