File: hardware/de0nano_cpu_card/sheets/level_shifters.kicad_sch (KiCad schematic)
At the start: 33 parts, among them J2 EXP_HEADER_2x11, U1 SN74LVC8T245, U2 SN74LVC8T245, U3 SN74LVC8T245, U4 SN74LVC8T245, U5 SN74LVC8T245, U6 SN74LVC8T245

Commit message: Routing done
Parts:
- removed R25, R26, R27: 10k, Resistor_SMD:R_0603_1608Metric, symbol Device:R
- added C21, C22, C23, C24: 100nF, Capacitor_SMD:C_0603_1608Metric, symbol Device:C
- added U8, U9: SN74LVC8T245, Package_SO:TSSOP-24_4.4x7.8mm_P0.65mm, symbol Logic_LevelTranslator:SN74LVC8T245
Connections:
- net U4_SPARE_B7 is gone; now on net GND: U4.15 (B7)
- net U4_SPARE_B8 is gone; now on net GND: U4.14 (B8)
- net +3V3: now also C21.1, C23.1, U8.1 (V_{CCA}), U8.2 (DIR), U9.1 (V_{CCA})
- net +5V: now also C22.1, C24.1, U8.23 (V_{CCB}), U8.24 (V_{CCB}), U9.23 (V_{CCB}), U9.24 (V_{CCB})
- net BP_LC: now also U9.21 (B1); no longer U4.21 (B1)
- net BP_N[0]: now also U8.15 (B7); no longer U2.15 (B7)
- net BP_N[1]: now also U8.16 (B6); no longer U2.16 (B6)
- net BP_N[2]: now also U8.17 (B5); no longer U2.17 (B5)
- net BP_Q: now also U8.14 (B8); no longer U2.14 (B8)
- net BP_nINT: now also U9.20 (B2); no longer U4.20 (B2)
- net BUF_nOE: now also U8.22 (~{OE})
- net GND: now also U2.10 (A8), U2.7 (A5), U2.8 (A6), U2.9 (A7), U4.16 (B6), U4.20 (B2), U4.21 (B1), C21.2, C22.2, C23.2, C24.2, U8.11 (GND), U8.12 (GND), U8.13 (GND), U8.3 (A1), U8.4 (A2), U8.5 (A3), U8.6 (A4), U9.11 (GND), U9.12 (GND), U9.13 (GND), U9.14 (B8), U9.15 (B7), U9.16 (B6), U9.17 (B5), U9.18 (B4), U9.19 (B3), U9.2 (DIR), U9.22 (~{OE})
- net LC: now also U9.3 (A1); no longer U4.3 (A1)
- net N[0]: now also U8.9 (A7); no longer U2.9 (A7)
- net N[1]: now also U8.8 (A6); no longer U2.8 (A6)
- net N[2]: now also U8.7 (A5); no longer U2.7 (A5)
- net Q: now also U8.10 (A8); no longer U2.10 (A8)
- net U4_SPARE_B6: no longer U4.16 (B6)
- net nINT: now also U9.4 (A2); no longer U4.4 (A2)
- no-connect marks 8 -> 24
Other:
- moved on the sheet: C10, C11, C12, C13, J2, U5, U6
