File: hardware/de0nano_cpu_card/sheets/power.kicad_sch (KiCad schematic)
At the start: 0 parts

Commit message: Wire up all 7 schematic sheets with real nets
All architecture/sourcing decisions were already resolved; this wires
them into the actual schematic, generated from docs/cs1800.qsf and the
other docs/ files via a small purpose-built generator (tools/) rather
than hand-placing ~400 pins in the GUI:

- backplane_connector: DIN41617 31p + 13 pull-up resistors per the
  backplane pinout's *1/*2 notes
- level_shifters: all 6 SN74LVC8T245 (4 backplane + 2 future-expansion),
  DIR/OE strapping per the power-up-safe defaults in backplane_notes.md,
  plus the future-expansion 2x11 header that was previously only
  documented, not placed
- fpga_header: both DE0-Nano GPIO headers (JP1/JP2), every pin from
  cs1800.qsf, VCC3P3 wired as the board's +3V3 source
- power: backplane 5V feed header, bulk cap, PWR_FLAGs
- pico_w_bridge: Pico-W module, UART0/UART1 routing, 8 spare GPIO,
  RUN pull-up, VSYS back-feed Schottky diode
- rs232: MAX3232 (channel 1 only) + DB9, charge-pump caps
- frontpanel_io: 4 LEDs w/ series resistors, 3 switches + 3 buttons w/
  pull-ups

kicad-cli sch erc on the full hierarchy: 0 errors, 3 known/benign
warnings (custom DIN41617 footprint not drawn yet; 2 cosmetic
lib_symbol_mismatch notices on the extends-based symbols). pcb drc on
the still-placeholder board outline: 0 violations.

Co-Authored-By: Claude Sonnet 5 <noreply@anthropic.com>
Parts:
- added C1: 100uF_LowESR, Capacitor_SMD:C_1210_3225Metric, symbol Device:C
- added P1: DE0Nano_5V_feed, Connector_PinHeader_2.54mm:PinHeader_1x02_P2.54mm_Vertical, symbol Connector_Generic:Conn_01x02
Connections:
- new net +5V: C1.1, P1.1 (Pin_1)
- new net GND: C1.2, P1.2 (Pin_2)
