File: hardware/de0nano_cpu_card/sheets/power.kicad_sch (KiCad schematic)
At the start: 2 parts, among them P1 DE0Nano_5V_feed

Commit message: Add pull-ups/ties on spare channels and series resistors, per GUI review
The user reviewed the schematics in the KiCad GUI and manually
rearranged component layout on several sheets -- so these fixes are
applied as surgical patches to the current saved files (new
tools/patch_*.py scripts) rather than via the usual build_*.py
regeneration, which would have discarded that layout work. See the new
"don't just re-run build_*.py" section in tools/README.md for the
workflow this establishes going forward.

Electrical changes (level_shifters.kicad_sch):
- 10k pull-up to +5V on all 7 EXP_* future-expansion header input nets
- U4 (backplane IN chip) spare B-side channels (pins 14/15/16): pulled
  out of no_connect, 10k pull-up to +5V each
- U6 (future-expansion IN chip) spare B-side channel (pin 14): pulled
  out of no_connect, 10k pull-up to +5V
- U5 (future-expansion OUT chip) spare A-side channels (pins 7/8/9/10):
  pulled out of no_connect, hard-tied to GND (unused transceiver
  inputs, no resistor needed)

Electrical changes (fpga_header.kicad_sch):
- 10 ohm series resistors on TPA/TPB/nMRD/nMWR at the FPGA end, per
  backplane_notes.md's signal-integrity note (originally suggested
  33-47 ohm; user chose 10 ohm)

sch erc on the full hierarchy: 0 errors. New warnings are the expected
ones (pin_to_pin on the GND hard-ties -- that's what a hard tie looks
like to ERC). pcb drc: 0 violations.

Also includes the project files as resaved by KiCad 10's GUI during
the user's review pass (sheet_instances/project-settings expansion,
plus the user's own layout rearrangement on all 7 sheets), and
gitignores the .history/ directory KiCad 10's local version-history
feature creates.

Co-Authored-By: Claude Sonnet 5 <noreply@anthropic.com>
Changed lines of the file:
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@@
 	(wire
 		(pts
-			(xy 34.29 41.91) (xy 31.75 41.91)
+			(xy 33.02 41.91) (xy 34.29 41.91)
+		)
+		(stroke
+			(width 0)
+			(type default)
+		)
+	)
+	(wire
+		(pts
+			(xy 33.02 45.72) (xy 31.75 45.72)
 		)
 		(stroke
@@
 	(wire
 		(pts
-			(xy 110.49 39.37) (xy 110.49 41.91)
+			(xy 97.79 40.64) (xy 97.79 41.91)
+		)
+		(stroke
+			(width 0)
+			(type default)
+		)
+	)
+	(wire
+		(pts
+			(xy 143.51 40.64) (xy 129.54 40.64)
+		)
+		(stroke
+			(width 0)
+			(type default)
+		)
+	)
+	(wire
+		(pts
+			(xy 129.54 40.64) (xy 129.54 39.37)
 		)
 		(stroke
@@
 	(wire
 		(pts
-			(xy 129.54 39.37) (xy 129.54 41.91)
+			(xy 110.49 40.64) (xy 110.49 39.37)
+		)
+		(stroke
+			(width 0)
+			(type default)
+		)
+	)
+	(wire
+		(pts
+			(xy 33.02 45.72) (xy 33.02 41.91)
+		)
+		(stroke
+			(width 0)
+			(type default)
+		)
+	)
+	(wire
+		(pts
+			(xy 97.79 40.64) (xy 110.49 40.64)
 		)
 		(stroke
@@
 	(global_label "+5V"
 		(shape input)
-		(at 110.49 41.91 90)
+		(at 97.79 41.91 90)
 		(effects
 			(font
@@
 		)
 		(property "Intersheetrefs" "${INTERSHEET_REFS}"
-			(at 110.49 41.91 0)
+			(at 97.79 41.91 0)
 			(hide yes)
 			(show_name no)
@@
 	(global_label "+3V3"
 		(shape input)
-		(at 129.54 41.91 90)
+		(at 143.51 40.64 90)
 		(effects
 			(font
@@
 		)
 		(property "Intersheetrefs" "${INTERSHEET_REFS}"
-			(at 129.54 41.91 0)
+			(at 143.51 40.64 0)
 			(hide yes)
 			(show_name no)
@@
 		(pin "1"
 		)
+		(instances
+			(project "de0nano_cpu_card"
+				(path "/0daab69e-2257-45dd-abd7-efbe947cce3e/8b002943-6b27-46a8-b3d0-f29a8b6e36ed"
+					(reference "#PWR")
+					(unit 1)
+				)
+			)
+		)
 	)
 	(symbol
@@
 		(pin "1"
 		)
+		(instances
+			(project "de0nano_cpu_card"
+				(path "/0daab69e-2257-45dd-abd7-efbe947cce3e/8b002943-6b27-46a8-b3d0-f29a8b6e36ed"
+					(reference "PF2")
+					(unit 1)
+				)
+			)
+		)
 	)
 	(symbol
 		(lib_id "power:GND")
-		(at 31.75 41.91 0)
+		(at 31.75 45.72 0)
 		(unit 1)
 		(body_style 1)
@@
 		(dnp no)
 		(property "Reference" "#PWR"
-			(at 31.75 41.91 0)
+			(at 31.75 45.72 0)
 			(hide yes)
 			(show_name no)
@@
 		)
 		(property "Value" "GND"
-			(at 31.75 39.37 0)
+			(at 31.75 43.18 0)
 			(show_name no)
 			(do_not_autoplace no)
@@
 		)
 		(property "Footprint" ""
-			(at 31.75 41.91 0)
+			(at 31.75 45.72 0)
 			(show_name no)
 			(do_not_autoplace no)
@@
 		)
 		(property "Datasheet" ""
-			(at 31.75 41.91 0)
+			(at 31.75 45.72 0)
 			(show_name no)
 			(do_not_autoplace no)
@@
 		)
 		(property "Description" ""
-			(at 31.75 41.91 0)
+			(at 31.75 45.72 0)
 			(show_name no)
 			(do_not_autoplace no)
@@
 		)
 		(pin "1"
+		)
+		(instances
+			(project "de0nano_cpu_card"
+				(path "/0daab69e-2257-45dd-abd7-efbe947cce3e/8b002943-6b27-46a8-b3d0-f29a8b6e36ed"
+					(reference "#PWR")
+					(unit 1)
+				)
+			)
 		)
 	)
@@
 		(pin "2"
 		)
+		(instances
+			(project "de0nano_cpu_card"
+				(path "/0daab69e-2257-45dd-abd7-efbe947cce3e/8b002943-6b27-46a8-b3d0-f29a8b6e36ed"
+					(reference "C1")
+					(unit 1)
+				)
+			)
+		)
 	)
 	(symbol
@@
 		(pin "2"
 		)
+		(instances
+			(project "de0nano_cpu_card"
+				(path "/0daab69e-2257-45dd-abd7-efbe947cce3e/8b002943-6b27-46a8-b3d0-f29a8b6e36ed"
+					(reference "P1")
+					(unit 1)
+				)
+			)
+		)
 	)
 	(symbol
@@
 		(pin "1"
 		)
+		(instances
+			(project "de0nano_cpu_card"
+				(path "/0daab69e-2257-45dd-abd7-efbe947cce3e/8b002943-6b27-46a8-b3d0-f29a8b6e36ed"
+					(reference "PF1")
+					(unit 1)
+				)
+			)
+		)
 	)
 	(symbol
@@
 		(pin "1"
 		)
+		(instances
+			(project "de0nano_cpu_card"
+				(path "/0daab69e-2257-45dd-abd7-efbe947cce3e/8b002943-6b27-46a8-b3d0-f29a8b6e36ed"
+					(reference "#PWR")
+					(unit 1)
+				)
+			)
+		)
 	)
 	(symbol
@@
 		(pin "1"
 		)
-	)
+		(instances
+			(project "de0nano_cpu_card"
+				(path "/0daab69e-2257-45dd-abd7-efbe947cce3e/8b002943-6b27-46a8-b3d0-f29a8b6e36ed"
+					(reference "#PWR")
+					(unit 1)
+				)
+			)
+		)
+	)
