File: hardware/de0nano_cpu_card/sheets/rs232.kicad_sch (KiCad schematic)
At the start: 0 parts

Commit message: Wire up all 7 schematic sheets with real nets
All architecture/sourcing decisions were already resolved; this wires
them into the actual schematic, generated from docs/cs1800.qsf and the
other docs/ files via a small purpose-built generator (tools/) rather
than hand-placing ~400 pins in the GUI:

- backplane_connector: DIN41617 31p + 13 pull-up resistors per the
  backplane pinout's *1/*2 notes
- level_shifters: all 6 SN74LVC8T245 (4 backplane + 2 future-expansion),
  DIR/OE strapping per the power-up-safe defaults in backplane_notes.md,
  plus the future-expansion 2x11 header that was previously only
  documented, not placed
- fpga_header: both DE0-Nano GPIO headers (JP1/JP2), every pin from
  cs1800.qsf, VCC3P3 wired as the board's +3V3 source
- power: backplane 5V feed header, bulk cap, PWR_FLAGs
- pico_w_bridge: Pico-W module, UART0/UART1 routing, 8 spare GPIO,
  RUN pull-up, VSYS back-feed Schottky diode
- rs232: MAX3232 (channel 1 only) + DB9, charge-pump caps
- frontpanel_io: 4 LEDs w/ series resistors, 3 switches + 3 buttons w/
  pull-ups

kicad-cli sch erc on the full hierarchy: 0 errors, 3 known/benign
warnings (custom DIN41617 footprint not drawn yet; 2 cosmetic
lib_symbol_mismatch notices on the extends-based symbols). pcb drc on
the still-placeholder board outline: 0 violations.

Co-Authored-By: Claude Sonnet 5 <noreply@anthropic.com>
Parts:
- added C1, C2, C3, C4: 0.1uF, Capacitor_SMD:C_0603_1608Metric, symbol Device:C
- added J1: DB9_RS232, Connector_Dsub:DSUB-9_Pins_Horizontal_P2.77x2.54mm_EdgePinOffset9.40mm, symbol Connector:DE9_Pins
- added U1: MAX3232EIDR, Package_SO:SOIC-16_3.9x9.9mm_P1.27mm, symbol Interface_UART:MAX3232
Connections:
- new net +3V3: U1.16 (VCC)
- new net GND: C3.2, C4.2, J1.5, U1.15 (GND)
- new net MAX_C1N: C1.2, U1.3 (C1-)
- new net MAX_C1P: C1.1, U1.1 (C1+)
- new net MAX_C2N: C2.2, U1.5 (C2-)
- new net MAX_C2P: C2.1, U1.4 (C2+)
- new net MAX_VS+: C3.1, U1.2 (VS+)
- new net MAX_VS-: C4.1, U1.6 (VS-)
- new net PICO_UART1_RX: U1.12 (R1OUT)
- new net PICO_UART1_TX: U1.11 (T1IN)
- new net RS232_RXD: J1.2, U1.13 (R1IN)
- new net RS232_TXD: J1.3, U1.14 (T1OUT)
- no-connect marks 0 -> 10
