File: hardware/de0nano_cpu_card/sheets/rs232.kicad_sch (KiCad schematic)
At the start: 6 parts, among them J1 DB9_RS232, U1 MAX3232EIDR

Commit message: Add pull-ups/ties on spare channels and series resistors, per GUI review
The user reviewed the schematics in the KiCad GUI and manually
rearranged component layout on several sheets -- so these fixes are
applied as surgical patches to the current saved files (new
tools/patch_*.py scripts) rather than via the usual build_*.py
regeneration, which would have discarded that layout work. See the new
"don't just re-run build_*.py" section in tools/README.md for the
workflow this establishes going forward.

Electrical changes (level_shifters.kicad_sch):
- 10k pull-up to +5V on all 7 EXP_* future-expansion header input nets
- U4 (backplane IN chip) spare B-side channels (pins 14/15/16): pulled
  out of no_connect, 10k pull-up to +5V each
- U6 (future-expansion IN chip) spare B-side channel (pin 14): pulled
  out of no_connect, 10k pull-up to +5V
- U5 (future-expansion OUT chip) spare A-side channels (pins 7/8/9/10):
  pulled out of no_connect, hard-tied to GND (unused transceiver
  inputs, no resistor needed)

Electrical changes (fpga_header.kicad_sch):
- 10 ohm series resistors on TPA/TPB/nMRD/nMWR at the FPGA end, per
  backplane_notes.md's signal-integrity note (originally suggested
  33-47 ohm; user chose 10 ohm)

sch erc on the full hierarchy: 0 errors. New warnings are the expected
ones (pin_to_pin on the GND hard-ties -- that's what a hard tie looks
like to ERC). pcb drc: 0 violations.

Also includes the project files as resaved by KiCad 10's GUI during
the user's review pass (sheet_instances/project-settings expansion,
plus the user's own layout rearrangement on all 7 sheets), and
gitignores the .history/ directory KiCad 10's local version-history
feature creates.

Co-Authored-By: Claude Sonnet 5 <noreply@anthropic.com>
Other:
- moved on the sheet: C1
