File: hardware/de0nano_cpu_card/sheets/rs232.kicad_sch (KiCad schematic)
At the start: 6 parts, among them J1 DB9_RS232, U1 MAX3232EIDR

Commit message: Fix cross-sheet reference-designator collisions (required for PCB work)
Each build_*.py numbered its own parts independently (R1, C1, J1, U1,
etc. each starting fresh per sheet), which kicad-cli sch erc never
flagged -- ERC resolves connectivity by net name, not reference, so
duplicate refs across sheets are invisible to it. Only surfaced when
starting PCB work: `kicad-cli sch export netlist` warned about
annotation errors, and its (components) section showed 19 reference
names each silently mapping to 2-4 different real parts (89 components
total, e.g. "R1" meant three unrelated resistors on three sheets).

Fixed via tools/patch_reannotate_global.py: 60 references renumbered
to be globally unique, processed in root-sheet hierarchy order.
Required updating BOTH the visible (property "Reference" ...) field
and the (reference ...) inside each symbol's (instances ...) block --
the netlist exporter reads only the latter, so a first attempt that
touched just the property field silently had no effect on the
netlist. Both quirks documented in tools/README.md.

Verified: netlist's (components) section now has zero duplicate refs
(89 unique). sch erc: still 0 errors. pcb drc: still 0 violations.

Co-Authored-By: Claude Sonnet 5 <noreply@anthropic.com>
Parts:
- renumbered C1 to C16, C2 to C17, C3 to C18, C4 to C19, J1 to J5, U1 to U7
Changed lines of the file:
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@@
 		(in_pos_files yes)
 		(dnp no)
-		(property "Reference" "C4"
+		(property "Reference" "C19"
 			(at 139.7 84.17 0)
 			(show_name no)
@@
 			(project "de0nano_cpu_card"
 				(path "/0daab69e-2257-45dd-abd7-efbe947cce3e/06cb3957-3e2a-42f7-9aab-bec97b55ee82"
-					(reference "C4")
+					(reference "C19")
 					(unit 1)
 				)
@@
 		(in_pos_files yes)
 		(dnp no)
-		(property "Reference" "U1"
+		(property "Reference" "U7"
 			(at 100.33 53.69 0)
 			(show_name no)
@@
 			(project "de0nano_cpu_card"
 				(path "/0daab69e-2257-45dd-abd7-efbe947cce3e/06cb3957-3e2a-42f7-9aab-bec97b55ee82"
-					(reference "U1")
+					(reference "U7")
 					(unit 1)
 				)
@@
 		(in_pos_files yes)
 		(dnp no)
-		(property "Reference" "C2"
+		(property "Reference" "C17"
 			(at 139.7 24.48 0)
 			(show_name no)
@@
 			(project "de0nano_cpu_card"
 				(path "/0daab69e-2257-45dd-abd7-efbe947cce3e/06cb3957-3e2a-42f7-9aab-bec97b55ee82"
-					(reference "C2")
+					(reference "C17")
 					(unit 1)
 				)
@@
 		(in_pos_files yes)
 		(dnp no)
-		(property "Reference" "C1"
+		(property "Reference" "C16"
 			(at 45.72 23.21 0)
 			(show_name no)
@@
 			(project "de0nano_cpu_card"
 				(path "/0daab69e-2257-45dd-abd7-efbe947cce3e/06cb3957-3e2a-42f7-9aab-bec97b55ee82"
-					(reference "C1")
+					(reference "C16")
 					(unit 1)
 				)
@@
 		(in_pos_files yes)
 		(dnp no)
-		(property "Reference" "C3"
+		(property "Reference" "C18"
 			(at 59.69 84.17 0)
 			(show_name no)
@@
 			(project "de0nano_cpu_card"
 				(path "/0daab69e-2257-45dd-abd7-efbe947cce3e/06cb3957-3e2a-42f7-9aab-bec97b55ee82"
-					(reference "C3")
+					(reference "C18")
 					(unit 1)
 				)
@@
 		(in_pos_files yes)
 		(dnp no)
-		(property "Reference" "J1"
+		(property "Reference" "J5"
 			(at 219.71 53.69 0)
 			(show_name no)
@@
 			(project "de0nano_cpu_card"
 				(path "/0daab69e-2257-45dd-abd7-efbe947cce3e/06cb3957-3e2a-42f7-9aab-bec97b55ee82"
-					(reference "J1")
-					(unit 1)
-				)
+					(reference "J5")
+					(unit 1)
+				)
