File: hardware/de0nano_cpu_card/sheets/rs232.kicad_sch (KiCad schematic)
At the start: 6 parts, among them J5 DB9_RS232, U7 MAX3232EIDR

Commit message: more routing done. also done several pin swapping
Parts:
- added C20: 0.1uF, Capacitor_SMD:C_0603_1608Metric, symbol Device:C
Connections:
- net +3V3: now also C20.2
- net GND: now also U7.10 (T2IN), U7.8 (R2IN), C20.1
- no-connect marks 10 -> 8

Commit message: Routing done
Connections:
- net +3V3 renamed PICO_3V3
Changed lines of the file:
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@@
 	(wire
 		(pts
-			(xy 100.33 27.94) (xy 100.33 26.67)
+			(xy 100.33 25.4) (xy 100.33 27.94)
 		)
 		(stroke
@@
 	(wire
 		(pts
+			(xy 100.33 25.4) (xy 104.14 25.4)
+		)
+		(stroke
+			(width 0)
+			(type default)
+		)
+	)
+	(wire
+		(pts
 			(xy 74.93 25.4) (xy 74.93 26.67)
 		)
@@
 		)
 	)
-	(symbol
-		(lib_id "power:+3V3")
-		(at 100.33 26.67 0)
-		(unit 1)
-		(body_style 1)
-		(exclude_from_sim no)
-		(in_bom yes)
-		(on_board yes)
-		(in_pos_files yes)
-		(dnp no)
-		(property "Reference" "#PWR0154"
-			(at 100.33 26.67 0)
-			(hide yes)
-			(show_name no)
-			(do_not_autoplace no)
-			(effects
-				(font
-					(size 1.27 1.27)
-				)
-			)
-		)
-		(property "Value" "+3V3"
-			(at 100.33 24.13 0)
-			(show_name no)
-			(do_not_autoplace no)
-			(effects
-				(font
-					(size 1.27 1.27)
-				)
-			)
-		)
-		(property "Footprint" ""
-			(at 100.33 26.67 0)
-			(show_name no)
-			(do_not_autoplace no)
-			(effects
-				(font
-					(size 1.27 1.27)
-				)
-			)
-		)
-		(property "Datasheet" ""
-			(at 100.33 26.67 0)
-			(show_name no)
-			(do_not_autoplace no)
-			(effects
-				(font
-					(size 1.27 1.27)
-				)
-			)
-		)
-		(property "Description" ""
-			(at 100.33 26.67 0)
-			(show_name no)
-			(do_not_autoplace no)
-			(effects
-				(font
-					(size 1.27 1.27)
-				)
-			)
-		)
-		(pin "1"
-		)
-		(instances
-			(project "de0nano_cpu_card"
-				(path "/0daab69e-2257-45dd-abd7-efbe947cce3e/06cb3957-3e2a-42f7-9aab-bec97b55ee82"
-					(reference "#PWR0154")
-					(unit 1)
-				)
-			)
+	(global_label "PICO_3V3"
+		(shape input)
+		(at 104.14 25.4 90)
+		(effects
+			(font
+				(size 1.27 1.27)
+			)
+		)
+		(property "Intersheetrefs" "${INTERSHEET_REFS}"
+			(at 104.14 25.4 0)
+			(hide yes)
+			(show_name no)
+			(do_not_autoplace no)
+			(effects
+				(font
+					(size 1.27 1.27)
+				)
+			)
