File: hardware/de0nano_cpu_card/sheets/pico_w_bridge.kicad_sch (KiCad schematic)
At the start: 0 parts

Commit message: Sync docs/schematic skeleton with FT2232H -> Raspberry Pi Pico-W decision
Pico-W replaces the FT2232H dual-UART bridge (cheaper, fast enough for
2 simple UARTs, adds WiFi/telnet and spare GPIOs for free). Renamed the
placeholder schematic sheet accordingly and updated design_notes.md to
reflect the now-resolved backplane pinout, Eurocard floorplan, and
front-panel wiring, plus the new open items the Pico-W swap introduces
(antenna keepout, USB/backplane back-feed protection).

Co-Authored-By: Claude Sonnet 5 <noreply@anthropic.com>
Other:
- title: USB-Serial Bridge (FT2232H) -> UART Bridge (Raspberry Pi Pico-W)
Changed lines of the file:
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@@
 	(paper "A4")
 	(title_block
-		(title "USB-Serial Bridge (FT2232H)")
+		(title "UART Bridge (Raspberry Pi Pico-W)")
 		(date "2026-09-28")
 		(rev "A")

Commit message: Wire up all 7 schematic sheets with real nets
All architecture/sourcing decisions were already resolved; this wires
them into the actual schematic, generated from docs/cs1800.qsf and the
other docs/ files via a small purpose-built generator (tools/) rather
than hand-placing ~400 pins in the GUI:

- backplane_connector: DIN41617 31p + 13 pull-up resistors per the
  backplane pinout's *1/*2 notes
- level_shifters: all 6 SN74LVC8T245 (4 backplane + 2 future-expansion),
  DIR/OE strapping per the power-up-safe defaults in backplane_notes.md,
  plus the future-expansion 2x11 header that was previously only
  documented, not placed
- fpga_header: both DE0-Nano GPIO headers (JP1/JP2), every pin from
  cs1800.qsf, VCC3P3 wired as the board's +3V3 source
- power: backplane 5V feed header, bulk cap, PWR_FLAGs
- pico_w_bridge: Pico-W module, UART0/UART1 routing, 8 spare GPIO,
  RUN pull-up, VSYS back-feed Schottky diode
- rs232: MAX3232 (channel 1 only) + DB9, charge-pump caps
- frontpanel_io: 4 LEDs w/ series resistors, 3 switches + 3 buttons w/
  pull-ups

kicad-cli sch erc on the full hierarchy: 0 errors, 3 known/benign
warnings (custom DIN41617 footprint not drawn yet; 2 cosmetic
lib_symbol_mismatch notices on the extends-based symbols). pcb drc on
the still-placeholder board outline: 0 violations.

Co-Authored-By: Claude Sonnet 5 <noreply@anthropic.com>
Parts:
- added A1: RaspberryPi_Pico_W, Module:RaspberryPi_Pico_W_SMD_HandSolder, symbol MCU_Module:RaspberryPi_Pico_W
- added C1: 10uF_LowESR, Capacitor_SMD:C_1210_3225Metric, symbol Device:C
- added D1: 1N5817, Diode_SMD:D_SMA, symbol Device:D_Schottky
- added R1: 10k, Resistor_SMD:R_0603_1608Metric, symbol Device:R
Connections:
- new net +3V3: R1.1
- new net +5V: C1.1, D1.2 (A)
- new net GND: A1.13 (GND), A1.18 (GND), A1.23 (GND), A1.28 (GND), A1.3 (GND), A1.38 (GND), A1.8 (GND), C1.2
- new net PICO[0]: A1.19 (GPIO14)
- new net PICO[1]: A1.20 (GPIO15)
- new net PICO[2]: A1.21 (GPIO16)
- new net PICO[3]: A1.22 (GPIO17)
- new net PICO[4]: A1.24 (GPIO18)
- new net PICO[5]: A1.25 (GPIO19)
- new net PICO[6]: A1.26 (GPIO20)
- new net PICO[7]: A1.27 (GPIO21)
- new net PICO_RUN: A1.30 (RUN), R1.2
- new net PICO_UART1_RX: A1.7 (GPIO5)
- new net PICO_UART1_TX: A1.6 (GPIO4)
- new net PICO_VSYS: A1.39 (VSYS), D1.1 (K)
- new net UART0_RXD: A1.1 (GPIO0)
- new net UART0_TXD: A1.2 (GPIO1)
- no-connect marks 0 -> 19

Commit message: Mount Pico-W on socket headers instead of direct-solder
Needed so the Pico-W's own micro-USB port has room for a cable once
elevated above this board -- direct-soldering it would sit the module
right on the PCB surface with no clearance.

New footprint cs1800:RaspberryPi_Pico_W_SocketHeaders_2x1x20_P2.54mm
(tools/gen_pico_socket_fp.py): two 1x20 2.54mm-pitch socket rows,
17.78mm apart, matching genuine Pico/Pico W header spacing (cross-
checked against KiCad's own RaspberryPi_Pico_Common_THT footprint).
Pad numbering 1-20/21-40 matches the Pico's own pin numbers.

Noted in the BOM that the socket strips should be a tall/stacking-
height part, not low-profile -- the footprint only fixes pad
positions, actual USB-cable clearance is a part-sourcing choice.

sch erc: still 0 errors, same 2 cosmetic warnings as before.

Co-Authored-By: Claude Sonnet 5 <noreply@anthropic.com>
Parts:
- A1: footprint Module:RaspberryPi_Pico_W_SMD_HandSolder -> cs1800:RaspberryPi_Pico_W_SocketHeaders_2x1x20_P2.54mm
