File: hardware/de0nano_cpu_card/sheets/pico_w_bridge.kicad_sch (KiCad schematic)
At the start: 4 parts

Commit message: Fix cross-sheet reference-designator collisions (required for PCB work)
Each build_*.py numbered its own parts independently (R1, C1, J1, U1,
etc. each starting fresh per sheet), which kicad-cli sch erc never
flagged -- ERC resolves connectivity by net name, not reference, so
duplicate refs across sheets are invisible to it. Only surfaced when
starting PCB work: `kicad-cli sch export netlist` warned about
annotation errors, and its (components) section showed 19 reference
names each silently mapping to 2-4 different real parts (89 components
total, e.g. "R1" meant three unrelated resistors on three sheets).

Fixed via tools/patch_reannotate_global.py: 60 references renumbered
to be globally unique, processed in root-sheet hierarchy order.
Required updating BOTH the visible (property "Reference" ...) field
and the (reference ...) inside each symbol's (instances ...) block --
the netlist exporter reads only the latter, so a first attempt that
touched just the property field silently had no effect on the
netlist. Both quirks documented in tools/README.md.

Verified: netlist's (components) section now has zero duplicate refs
(89 unique). sch erc: still 0 errors. pcb drc: still 0 violations.

Co-Authored-By: Claude Sonnet 5 <noreply@anthropic.com>
Parts:
- renumbered C1 to C15, R1 to R32
Changed lines of the file:
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@@
 		(in_pos_files yes)
 		(dnp no)
-		(property "Reference" "C1"
+		(property "Reference" "C15"
 			(at 100.33 95.6 0)
 			(show_name no)
@@
 			(project "de0nano_cpu_card"
 				(path "/0daab69e-2257-45dd-abd7-efbe947cce3e/869c89e1-96aa-439b-bac8-8b2b26d1ef4c"
-					(reference "C1")
+					(reference "C15")
 					(unit 1)
 				)
@@
 		(in_pos_files yes)
 		(dnp no)
-		(property "Reference" "R1"
+		(property "Reference" "R32"
 			(at 180.34 95.6 0)
 			(show_name no)
@@
 			(project "de0nano_cpu_card"
 				(path "/0daab69e-2257-45dd-abd7-efbe947cce3e/869c89e1-96aa-439b-bac8-8b2b26d1ef4c"
-					(reference "R1")
+					(reference "R32")
 					(unit 1)
 				)
@@
 		(in_pos_files yes)
 		(dnp no)
-		(property "Reference" "PF1"
+		(property "Reference" "PF3"
 			(at 120.65 175.61 0)
 			(show_name no)
@@
 			(project "de0nano_cpu_card"
 				(path "/0daab69e-2257-45dd-abd7-efbe947cce3e/869c89e1-96aa-439b-bac8-8b2b26d1ef4c"
-					(reference "PF1")
-					(unit 1)
-				)
+					(reference "PF3")
+					(unit 1)
+				)
