File: hardware/de0nano_cpu_card/sheets/pico_w_bridge.kicad_sch (KiCad schematic)
At the start: 4 parts

Commit message: more routing done. also done several pin swapping
Parts:
- removed R32: 10k, Resistor_SMD:R_0603_1608Metric, symbol Device:R
Connections:
- net PICO[0]: now also A1.9 (GPIO6); no longer A1.19 (GPIO14)
- net PICO[1]: now also A1.10 (GPIO7); no longer A1.20 (GPIO15)
- net PICO[2]: now also A1.11 (GPIO8); no longer A1.21 (GPIO16)
- net PICO[3]: now also A1.12 (GPIO9); no longer A1.22 (GPIO17)
- net PICO[4]: now also A1.14 (GPIO10); no longer A1.24 (GPIO18)
- net PICO[5]: now also A1.15 (GPIO11); no longer A1.25 (GPIO19)
- net PICO[6]: now also A1.16 (GPIO12); no longer A1.26 (GPIO20)
- net PICO[7]: now also A1.17 (GPIO13); no longer A1.27 (GPIO21)
- net PICO_RUN: no longer names the net of A1.30 (RUN)
- no-connect marks 19 -> 20

Commit message: Routing done
Connections:
- net PICO_3V3: now reaches A1.36 (3V3)
- no-connect marks 20 -> 19
Changed lines of the file:
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@@
-	)
-	(no_connect
-		(at 146.05 102.87)
 	)
 	(no_connect
@@
 	(wire
 		(pts
+			(xy 146.05 100.33) (xy 146.05 102.87)
+		)
+		(stroke
+			(width 0)
+			(type default)
+		)
+	)
+	(wire
+		(pts
 			(xy 97.79 153.67) (xy 118.11 153.67)
 		)
@@
 		)
 	)
+	(global_label "PICO_3V3"
+		(shape input)
+		(at 146.05 100.33 90)
+		(effects
+			(font
+				(size 1.27 1.27)
+			)
+		)
+		(property "Intersheetrefs" "${INTERSHEET_REFS}"
+			(at 146.05 100.33 0)
+			(hide yes)
+			(show_name no)
+			(do_not_autoplace no)
+			(effects
+				(font
+					(size 1.27 1.27)
+				)
+			)
+		)
+	)
