File: hardware/de0nano_cpu_card/de0nano_cpu_card.kicad_pcb (KiCad board)
At the start: 2 copper layers, 100 x 160 mm, 0 parts

Commit message: PCB: real board outline, DE0-Nano reference, all 86 components placed
kicad-cli has no "update PCB from schematic" command, so getting the
schematic's components onto the board required building equivalent
tooling (tools/pcbgen.py + tools/build_pcb.py), parsing the schematic's
exported netlist for authoritative net/footprint data and real
.kicad_mod footprint files (staged in tools/fpstage/) for pad layout.

- Real 100x160mm Eurocard outline (was a generic placeholder rectangle)
- New cs1800:DE0Nano_Reference_Outline footprint: mechanical-only (NPTH
  mounting holes at the coordinates from design_notes.md Sec7, no
  copper pads -- the DE0-Nano connects via 2 ribbon cables, not by
  soldering to this board)
- All 86 real footprints placed (89 schematic components minus 3
  virtual PWR_FLAGs with no physical footprint), grouped roughly per
  Eurocard.md's left-to-right floorplan, with correct net assignments
  pulled straight from the netlist

This is a ROUGH placement only, by explicit agreement -- grouped, not
finely positioned. pcb drc: 0 electrical shorts, 309 unrouted
connections (expected, nothing routed yet), 77 remaining cosmetic/
mechanical placement warnings (silkscreen/courtyard overlaps, a couple
of edge-clearance nits) left for the user's real placement + routing
pass. Several PCB-specific generator quirks found and documented in
tools/README.md (net serialization after pcb upgrade, footprint
orientation assumptions, why the DE0-Nano reference has no reserved
clear zone).

Co-Authored-By: Claude Sonnet 5 <noreply@anthropic.com>
Parts:
- added A1: RaspberryPi_Pico_W, RaspberryPi_Pico_W_SocketHeaders_2x1x20_P2.54mm, F.Cu at (43.0, 50.0)
- added C1: 100pF, C_0603_1608Metric, F.Cu at (141.0, 95.0)
- added C10: 100nF, C_0603_1608Metric, F.Cu at (75.0, 3.00)
- added C11: 100nF, C_0603_1608Metric, F.Cu at (80.0, 3.00)
- added C12: 100nF, C_0603_1608Metric, F.Cu at (75.0, 18.0)
- added C13: 100nF, C_0603_1608Metric, F.Cu at (80.0, 18.0)
- added C14: 100uF_LowESR, C_1210_3225Metric, F.Cu at (110.0, 5.00)
- added C15: 10uF_LowESR, C_1210_3225Metric, F.Cu at (23.0, 56.0)
- added C16: 0.1uF, C_0603_1608Metric, F.Cu at (23.0, 15.0)
- added C17: 0.1uF, C_0603_1608Metric, F.Cu at (29.0, 15.0)
- added C18: 0.1uF, C_0603_1608Metric, F.Cu at (23.0, 21.0)
- added C19: 0.1uF, C_0603_1608Metric, F.Cu at (29.0, 21.0)
- added C2: 100nF, C_0603_1608Metric, F.Cu at (136.0, 3.00)
- added C3: 100nF, C_0603_1608Metric, F.Cu at (141.0, 3.00)
- added C4: 100nF, C_0603_1608Metric, F.Cu at (136.0, 18.0)
- added C5: 100nF, C_0603_1608Metric, F.Cu at (141.0, 18.0)
- added C6: 100nF, C_0603_1608Metric, F.Cu at (136.0, 33.0)
- added C7: 100nF, C_0603_1608Metric, F.Cu at (141.0, 33.0)
- added C8: 100nF, C_0603_1608Metric, F.Cu at (136.0, 48.0)
- added C9: 100nF, C_0603_1608Metric, F.Cu at (141.0, 48.0)
- added D1: 1N5817, D_SMA, F.Cu at (23.0, 50.0)
- added D2: LED_Green, LED_D3.0mm, F.Cu at (7.00, 5.00)
- added D3: LED_Yellow, LED_D3.0mm, F.Cu at (7.00, 12.0)
- added D4: LED_Red, LED_D3.0mm, F.Cu at (7.00, 19.0)
- added D5: LED_Red, LED_D3.0mm, F.Cu at (7.00, 26.0)
- added DE0NANO: DE0-Nano (reference), DE0Nano_Reference_Outline, F.Cu at (95.0, 12.0)
- added J1: DIN41617_31P, DIN41617_31P_Male_Angled, F.Cu at (154.0, 50.0)
- added J2: EXP_HEADER_2x11, PinHeader_2x11_P2.54mm_Vertical, F.Cu at (63.0, 55.0)
- added J3: GPIO_0_JP1, IDC-Header_2x20_P2.54mm_Vertical, F.Cu at (91.0, 50.0)
- added J4: GPIO_1_JP2, IDC-Header_2x20_P2.54mm_Vertical, F.Cu at (146.0, 50.0)
- added J5: DB9_RS232, DSUB-9_Pins_Horizontal_P2.77x2.54mm_EdgePinOffset9.40mm, F.Cu at (25.0, 30.0)
- added P1: DE0Nano_5V_feed, PinHeader_1x02_P2.54mm_Vertical, F.Cu at (100.0, 5.00)
- added R1: 10k, R_0603_1608Metric, F.Cu at (126.0, 80.0)
- added R10: 10k, R_0603_1608Metric, F.Cu at (130.0, 90.0)
- added R11: 10k, R_0603_1608Metric, F.Cu at (134.0, 90.0)
- added R12: 10k, R_0603_1608Metric, F.Cu at (138.0, 90.0)
- added R13: 10k, R_0603_1608Metric, F.Cu at (126.0, 95.0)
- added R14: 10k, R_0603_1608Metric, F.Cu at (126.0, 62.0)
- added R15: 10k, R_0603_1608Metric, F.Cu at (130.0, 62.0)
- added R16: 10k, R_0603_1608Metric, F.Cu at (134.0, 62.0)
- added R17: 10k, R_0603_1608Metric, F.Cu at (63.0, 35.0)
- added R18: 10k, R_0603_1608Metric, F.Cu at (69.0, 35.0)
- added R19: 10k, R_0603_1608Metric, F.Cu at (75.0, 35.0)
- added R2: 10k, R_0603_1608Metric, F.Cu at (130.0, 80.0)
- added R20: 10k, R_0603_1608Metric, F.Cu at (81.0, 35.0)
- added R21: 10k, R_0603_1608Metric, F.Cu at (63.0, 39.0)
- added R22: 10k, R_0603_1608Metric, F.Cu at (69.0, 39.0)
- added R23: 10k, R_0603_1608Metric, F.Cu at (75.0, 39.0)
- added R24: 10k, R_0603_1608Metric, F.Cu at (138.0, 62.0)
- added R25: 10k, R_0603_1608Metric, F.Cu at (126.0, 67.0)
- added R26: 10k, R_0603_1608Metric, F.Cu at (130.0, 67.0)
- added R27: 10k, R_0603_1608Metric, F.Cu at (81.0, 39.0)
- added R28: 10, R_0603_1608Metric, F.Cu at (134.0, 67.0)
- added R29: 10, R_0603_1608Metric, F.Cu at (138.0, 67.0)
- added R3: 10k, R_0603_1608Metric, F.Cu at (134.0, 80.0)
- added R30: 10, R_0603_1608Metric, F.Cu at (126.0, 72.0)
- added R31: 10, R_0603_1608Metric, F.Cu at (130.0, 72.0)
- added R32: 10k, R_0603_1608Metric, F.Cu at (23.0, 62.0)
- added R4: 10k, R_0603_1608Metric, F.Cu at (138.0, 80.0)
- added R5: 10k, R_0603_1608Metric, F.Cu at (126.0, 85.0)
- added R6: 10k, R_0603_1608Metric, F.Cu at (130.0, 85.0)
- added R7: 10k, R_0603_1608Metric, F.Cu at (134.0, 85.0)
- added R8: 10k, R_0603_1608Metric, F.Cu at (138.0, 85.0)
- added R9: 10k, R_0603_1608Metric, F.Cu at (126.0, 90.0)
- added R_D1: 220, R_0603_1608Metric, F.Cu at (14.0, 5.00)
- added R_D2: 220, R_0603_1608Metric, F.Cu at (14.0, 12.0)
- added R_D3: 220, R_0603_1608Metric, F.Cu at (14.0, 19.0)
- added R_D4: 220, R_0603_1608Metric, F.Cu at (14.0, 26.0)
- added R_SW1: 10k, R_0603_1608Metric, F.Cu at (14.0, 38.0)
- added R_SW2: 10k, R_0603_1608Metric, F.Cu at (14.0, 45.0)
- added R_SW3: 10k, R_0603_1608Metric, F.Cu at (14.0, 52.0)
- added R_SW4: 10k, R_0603_1608Metric, F.Cu at (14.0, 59.0)
- added R_SW5: 10k, R_0603_1608Metric, F.Cu at (14.0, 66.0)
- added R_SW6: 10k, R_0603_1608Metric, F.Cu at (14.0, 73.0)
- added SW1: Rocker_run/halt, PinHeader_1x02_P2.54mm_Vertical, F.Cu at (7.00, 38.0)
- added SW2: Rocker_dog_off, PinHeader_1x02_P2.54mm_Vertical, F.Cu at (7.00, 45.0)
- added SW3: Rocker_LC_off, PinHeader_1x02_P2.54mm_Vertical, F.Cu at (7.00, 52.0)
- added SW4: Button_step, PinHeader_1x02_P2.54mm_Vertical, F.Cu at (7.00, 59.0)
- added SW5: Button_reset, PinHeader_1x02_P2.54mm_Vertical, F.Cu at (7.00, 66.0)
- added SW6: Button_qef4, PinHeader_1x02_P2.54mm_Vertical, F.Cu at (7.00, 73.0)
- added U1: SN74LVC8T245, TSSOP-24_4.4x7.8mm_P0.65mm, F.Cu at (126.0, 5.00)
- added U2: SN74LVC8T245, TSSOP-24_4.4x7.8mm_P0.65mm, F.Cu at (126.0, 20.0)
- added U3: SN74LVC8T245, TSSOP-24_4.4x7.8mm_P0.65mm, F.Cu at (126.0, 35.0)
- added U4: SN74LVC8T245, TSSOP-24_4.4x7.8mm_P0.65mm, F.Cu at (126.0, 50.0)
- added U5: SN74LVC8T245, TSSOP-24_4.4x7.8mm_P0.65mm, F.Cu at (65.0, 5.00)
- added U6: SN74LVC8T245, TSSOP-24_4.4x7.8mm_P0.65mm, F.Cu at (65.0, 20.0)
- added U7: MAX3232EIDR, SOIC-16_3.9x9.9mm_P1.27mm, F.Cu at (25.0, 9.00)
Other:
- board size 100 x 160 mm -> 160 x 100 mm
- board text added: "CS1800 DE0-Nano CPU Card -- ROUGH PLACEMENT, not routed. Front panel at X=0 (left), backplane connector at X=160 (right). See docs/design_notes.md Sec7 / Eurocard.md for the intended floorplan."
- board text removed: "PLACEHOLDER OUTLINE 100 x 160 mm - single Eurocard depth. CONFIRM 'double slot' width/depth + DIN41617 connector position against the existing CS1800 backplane/rack before routing."
