File: hardware/de0nano_cpu_card/de0nano_cpu_card.kicad_pcb (KiCad board)
At the start: 2 copper layers, 160 x 100 mm, 87 parts, among them J1 DIN41617_31P, J2 EXP_HEADER_2x11, J3 GPIO_0_JP1, J4 GPIO_1_JP2, J5 DB9_RS232, P1 DE0Nano_5V_feed, SW1 Rocker_run/halt, SW2 Rocker_dog_off, SW3 Rocker_LC_off, SW4 Button_step, SW5 Button_reset, SW6 Button_qef4, U1 SN74LVC8T245, U2 SN74LVC8T245, U3 SN74LVC8T245, U4 SN74LVC8T245, U5 SN74LVC8T245, U6 SN74LVC8T245, U7 MAX3232EIDR

Commit message: Add 2 front-panel mounting holes on the board's left edge
Plain NPTH, 2.8mm drill, new generic cs1800:MountingHole_2.8mm footprint
(not tied to any connector/part, reusable for future mechanical-only
holes). Placed at (3.6, 5.5) and (3.6, 94.5) mm per the user's panel
measurements: 3.6mm from the left board edge, 5.5mm from top/bottom
edge, 89mm apart.

pcb drc: still 0 electrical shorts, 309 unrouted, 73 cosmetic warnings.

Co-Authored-By: Claude Sonnet 5 <noreply@anthropic.com>
Parts:
- added MH1: Front panel mounting hole, MountingHole_2.8mm, F.Cu at (3.60, 5.50)
- added MH2: Front panel mounting hole, MountingHole_2.8mm, F.Cu at (3.60, 94.5)
