File: hardware/de0nano_cpu_card/de0nano_cpu_card.kicad_pcb (KiCad board)
At the start: 2 copper layers, 160 x 100 mm, 89 parts, among them J1 DIN41617_31P, J2 EXP_HEADER_2x11, J3 GPIO_0_JP1, J4 GPIO_1_JP2, J5 DB9_RS232, P1 DE0Nano_5V_feed, SW1 Rocker_run/halt, SW2 Rocker_dog_off, SW3 Rocker_LC_off, SW4 Button_step, SW5 Button_reset, SW6 Button_qef4, U1 SN74LVC8T245, U2 SN74LVC8T245, U3 SN74LVC8T245, U4 SN74LVC8T245, U5 SN74LVC8T245, U6 SN74LVC8T245, U7 MAX3232EIDR

Commit message: Fixed mounting holes and backplane connector location
Parts:
- moved J4 198.9 mm to (267.8, 207.3)
- moved J1 186.6 mm to (286.0, 181.9)
- moved A1 165.0 mm to (178.3, 144.4)
- moved C10 165.0 mm to (210.3, 97.4)
- moved C11 165.0 mm to (215.3, 97.4)
- moved C12 165.0 mm to (210.3, 112.4)
- moved C13 165.0 mm to (215.3, 112.4)
- moved C14 165.0 mm to (245.3, 99.4)
- moved C15 165.0 mm to (158.3, 150.4)
- moved C16 165.0 mm to (158.3, 109.4)
- moved C17 165.0 mm to (164.3, 109.4)
- moved C18 165.0 mm to (158.3, 115.4)
- moved C19 165.0 mm to (164.3, 115.4)
- moved D1 165.0 mm to (158.3, 144.4)
- moved D2 165.0 mm to (142.3, 99.4)
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Other:
- board text added: "CS1800 DE0-Nano CPU Card"
- board text removed: "CS1800 DE0-Nano CPU Card -- ROUGH PLACEMENT, not routed. Front panel at X=0 (left), backplane connector at X=160 (right). See docs/design_notes.md Sec7 / Eurocard.md for the intended floorplan."

Commit message: placement optimalization process
Parts:
- MH1, MH2: value Front panel mounting hole -> f
- moved J4 111.2 mm to (195.4, 122.8)
- moved J2 102.2 mm to (214.1, 48.5)
- moved U7 77.9 mm to (157.1, 181.3)
- moved C16 69.9 mm to (142.9, 177.6)
- moved C17 69.9 mm to (148.9, 177.6)
- moved C18 69.9 mm to (142.9, 183.6)
- moved C19 69.9 mm to (148.9, 183.6)
- moved R27 69.5 mm to (201.8, 65.5), turned to -90 degrees
- moved R23 68.7 mm to (200.2, 65.5), turned to -90 degrees
- moved R22 68.2 mm to (198.7, 65.5), turned to -90 degrees
- moved R21 67.9 mm to (197.2, 65.5), turned to -90 degrees
- moved R20 67.2 mm to (195.6, 65.5), turned to -90 degrees
- moved R19 66.0 mm to (194.1, 65.5), turned to -90 degrees
- moved R18 65.0 mm to (192.6, 65.4), turned to -90 degrees
- moved C2 65.0 mm to (275.8, 32.6)
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
Commit message: placement OK. Started routing
Parts:
- moved U1 125.0 mm to (273.4, 161.3)
- moved C2 123.8 mm to (271.0, 156.3)
- moved C3 123.8 mm to (275.8, 156.2), turned to 180 degrees
- moved U2 101.8 mm to (273.3, 151.1)
- moved C5 98.6 mm to (275.7, 146.1), turned to 180 degrees
- moved C4 98.6 mm to (271.0, 146.1)
- moved C1 93.8 mm to (282.4, 112.5), turned to 180 degrees
- moved C10 88.0 mm to (204.1, 136.6), turned to 90 degrees
- moved C11 83.1 mm to (204.1, 131.7), turned to -90 degrees
- moved C12 81.3 mm to (216.7, 137.0), turned to 90 degrees
- moved U5 80.7 mm to (209.1, 134.2), turned to 90 degrees
- moved R2 76.5 mm to (282.4, 110.9)
- moved R1 75.9 mm to (282.4, 109.3)
- moved U6 75.6 mm to (221.8, 134.5), turned to 90 degrees
- moved C13 74.6 mm to (216.7, 131.9), turned to -90 degrees
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Routing:
- net GND: track 0.00 -> 873.7 mm
- net +5V: track 0.00 -> 264.8 mm
- net nDMA_OUT: track 0.00 -> 40.2 mm
- net nDMA_IN: track 0.00 -> 38.5 mm
- net nCLEAR: track 0.00 -> 37.6 mm
- net nWAIT: track 0.00 -> 35.8 mm
- net EX_IN[1]: track 0.00 -> 35.0 mm
- net nEF[3]: track 0.00 -> 33.2 mm
- net EXP_EX_IN[0]: track 0.00 -> 32.7 mm, vias 0 -> 1
- net EXP_nDMA_IN: track 0.00 -> 31.0 mm, vias 0 -> 1
- net EXP_EX_IN[1]: track 0.00 -> 30.9 mm, vias 0 -> 1
- net EX_IN[0]: track 0.00 -> 30.7 mm
- net EXP_nDMA_OUT: track 0.00 -> 30.3 mm, vias 0 -> 1
- net EXP_CS[0]: track 0.00 -> 30.1 mm
- net EXP_nCLEAR: track 0.00 -> 29.6 mm, vias 0 -> 1
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Other:
- board text added: "CS1800 DE0-Nano CPU Card Leon Hiemstra Oct-2026"
- board text removed: "CS1800 DE0-Nano CPU Card"

Commit message: more routing done. also done several pin swapping
Parts:
- removed R32: 10k, R_0603_1608Metric
- added C20: 0.1uF, Capacitor_SMD:C_0603_1608Metric, F.Cu at (154.5, 161.5)
- A1: footprint RaspberryPi_Pico_W_SocketHeaders_2x1x20_P2.54mm -> cs1800:RaspberryPi_Pico_W_SocketHeaders_2x1x20_P2.54mm
- U7: footprint SOIC-16_3.9x9.9mm_P1.27mm -> Package_SO:SOIC-16_3.9x9.9mm_P1.27mm
- moved R_D3 3.20 mm to (143.1, 122.1), turned to 180 degrees
- moved R_SW5 2.54 mm to (147.4, 144.3)
- moved SW5 2.54 mm to (144.7, 143.5)
- moved R_D1 2.37 mm to (143.0, 113.9), turned to 180 degrees
- moved R_SW6 1.49 mm to (141.2, 144.2)
- moved SW6 1.49 mm to (138.6, 143.4)
- moved R_SW2 1.24 mm to (149.0, 129.0), turned to 90 degrees
- moved R_SW3 1.16 mm to (154.4, 129.1), turned to 90 degrees
- moved R_D4 0.89 mm to (143.2, 132.1), turned to 180 degrees
- moved R_D2 0.81 mm to (143.0, 118.0), turned to 180 degrees
- moved C19 0.50 mm to (155.2, 163.9)
- moved U7 0.11 mm to (161.3, 163.9)
- moved A1 0.09 mm to (182.1, 150.3)
Connections:
- A1 pad 10: unconnected-(A1-GPIO7-Pad10) -> PICO[1]
- A1 pad 11: unconnected-(A1-GPIO8-Pad11) -> PICO[2]
- A1 pad 12: unconnected-(A1-GPIO9-Pad12) -> PICO[3]
- A1 pad 14: unconnected-(A1-GPIO10-Pad14) -> PICO[4]
- A1 pad 15: unconnected-(A1-GPIO11-Pad15) -> PICO[5]
- A1 pad 16: unconnected-(A1-GPIO12-Pad16) -> PICO[6]
- A1 pad 17: unconnected-(A1-GPIO13-Pad17) -> PICO[7]
- A1 pad 19: PICO[0] -> unconnected-(A1-GPIO14-Pad19)
- A1 pad 20: PICO[1] -> unconnected-(A1-GPIO15-Pad20)
- A1 pad 21: PICO[2] -> unconnected-(A1-GPIO16-Pad21)
- A1 pad 22: PICO[3] -> unconnected-(A1-GPIO17-Pad22)
- A1 pad 24: PICO[4] -> unconnected-(A1-GPIO18-Pad24)
- A1 pad 25: PICO[5] -> unconnected-(A1-GPIO19-Pad25)
- A1 pad 26: PICO[6] -> unconnected-(A1-GPIO20-Pad26)
- A1 pad 27: PICO[7] -> unconnected-(A1-GPIO21-Pad27)
- A1 pad 30: PICO_RUN -> unconnected-(A1-RUN-Pad30)
- A1 pad 9: unconnected-(A1-GPIO6-Pad9) -> PICO[0]
- U7 pad 10: unconnected-(U7-T2IN-Pad10) -> GND
- U7 pad 8: unconnected-(U7-R2IN-Pad8) -> GND
Routing:
- net +3V3: track 3.93 -> 261.9 mm, vias 0 -> 2
- net BUT_step: track 0.00 -> 103.8 mm, vias 0 -> 1
- net SW_halt: track 0.00 -> 96.1 mm, vias 0 -> 1
- net LED2_execute: track 0.00 -> 90.0 mm
- net LED1_fetch: track 0.00 -> 87.8 mm
- net LED3_interrupt: track 0.00 -> 85.5 mm
- net SW_dog: track 0.00 -> 82.3 mm, vias 0 -> 1
- net SW_LC_off: track 0.00 -> 78.5 mm, vias 0 -> 1
- net LED4_Q: track 0.00 -> 75.7 mm
- net BUT_qef4: track 0.00 -> 74.9 mm
- net BUT_reset: track 0.00 -> 68.1 mm
- net PICO_UART1_RX: track 0.00 -> 47.2 mm, vias 0 -> 2
- net PICO_UART1_TX: track 0.00 -> 41.4 mm, vias 0 -> 2
- net PICO[7]: track 0.00 -> 32.1 mm
- net UART0_TXD: track 0.00 -> 31.8 mm
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
Commit message: Routing done
Parts:
- removed R24, R25, R26: 10k, R_0603_1608Metric
- added C21: 100nF, Capacitor_SMD:C_0603_1608Metric, F.Cu at (268.5, 168.1)
- added C22: 100nF, Capacitor_SMD:C_0603_1608Metric, F.Cu at (273.2, 168.1)
- added C23: 100nF, Capacitor_SMD:C_0603_1608Metric, F.Cu at (268.7, 113.1)
- added C24: 100nF, Capacitor_SMD:C_0603_1608Metric, F.Cu at (273.6, 113.1)
- added U8: SN74LVC8T245, Package_SO:TSSOP-24_4.4x7.8mm_P0.65mm, F.Cu at (270.9, 173.1)
- added U9: SN74LVC8T245, Package_SO:TSSOP-24_4.4x7.8mm_P0.65mm, F.Cu at (271.1, 118.0)
- U2, U4: footprint TSSOP-24_4.4x7.8mm_P0.65mm -> Package_SO:TSSOP-24_4.4x7.8mm_P0.65mm
- moved U2 23.0 mm to (271.1, 128.2)
- moved C5 23.0 mm to (273.4, 123.2)
- moved C4 23.0 mm to (268.7, 123.2)
- moved C6 22.2 mm to (268.5, 157.9)
- moved C7 22.2 mm to (273.3, 157.9)
- moved U4 22.2 mm to (270.9, 162.9)
- moved R16 14.2 mm to (274.3, 135.4), turned to -90 degrees
- moved R15 13.0 mm to (272.7, 135.3), turned to -90 degrees
- moved C9 12.1 mm to (273.5, 137.7)
- moved U3 12.1 mm to (271.0, 142.7)
- moved C8 12.1 mm to (268.6, 137.7)
- moved R14 12.0 mm to (265.6, 139.4)
- moved C2 8.81 mm to (268.6, 147.8)
- moved C3 8.81 mm to (273.4, 147.8)
- moved U1 8.81 mm to (271.0, 152.8)
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Connections:
- A1 pad 36: unconnected-(A1-3V3-Pad36) -> PICO_3V3
- C20 pad 2: +3V3 -> PICO_3V3
- U2 pad 10: Q -> GND
- U2 pad 14: BP_Q -> unconnected-(U2-B8-Pad14)
- U2 pad 15: BP_N[0] -> unconnected-(U2-B7-Pad15)
- U2 pad 16: BP_N[1] -> unconnected-(U2-B6-Pad16)
- U2 pad 17: BP_N[2] -> unconnected-(U2-B5-Pad17)
- U2 pad 7: N[2] -> GND
- U2 pad 8: N[1] -> GND
- U2 pad 9: N[0] -> GND
- U4 pad 14: U4_SPARE_B8 -> GND
- U4 pad 15: U4_SPARE_B7 -> GND
- U4 pad 16: U4_SPARE_B6 -> GND
- U4 pad 20: BP_nINT -> GND
- U4 pad 21: BP_LC -> GND
- U4 pad 3: LC -> unconnected-(U4-A1-Pad3)
- U4 pad 4: nINT -> unconnected-(U4-A2-Pad4)
- U7 pad 16: +3V3 -> PICO_3V3
Routing:
- net GND: track 889.4 -> 1065.9 mm, vias 0 -> 6
- net +5V: track 264.3 -> 424.5 mm, vias 0 -> 9
- net +3V3: track 261.9 -> 379.9 mm, vias 2 -> 10
- net BUF_nOE: track 0.00 -> 95.2 mm, vias 0 -> 4
- net BP_ADDR[7]: track 0.00 -> 32.9 mm, vias 0 -> 1
- net BP_ADDR[6]: track 0.00 -> 28.9 mm, vias 0 -> 1
- net PICO_3V3: track 0.00 -> 27.3 mm, vias 0 -> 1
- net BP_ADDR[5]: track 0.00 -> 24.8 mm, vias 0 -> 1
- net BP_DATA[7]: track 0.00 -> 24.5 mm
- net DATA_nOE: track 0.00 -> 24.3 mm
- net BP_DATA[5]: track 0.00 -> 22.0 mm
- net BP_ADDR[4]: track 0.00 -> 20.8 mm, vias 0 -> 1
- net ADDR[0]: track 0.00 -> 20.6 mm
- net BP_ADDR[1]: track 0.00 -> 20.4 mm
- net BP_DATA[6]: track 0.00 -> 19.9 mm
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
Commit message: Added GND via-stitching and GND planes
Parts:
- moved R3 0.87 mm to (282.6, 125.3)
Routing:
- net GND: track 1065.9 -> 1696.3 mm, vias 6 -> 60
- net +5V: track 424.5 -> 429.0 mm
- net EX_OUT[1]: track 22.6 -> 24.2 mm
- net CS[1]: track 19.9 -> 21.4 mm
- net ADDR[0]: track 20.6 -> 19.0 mm
- net EX_OUT[0]: track 18.2 -> 19.7 mm
- net +3V3: track 379.9 -> 381.3 mm
- net CS[0]: track 15.5 -> 17.0 mm
- added copper zone on B.Cu, net GND
- added copper zone on F.Cu, net GND
