File: hardware/de0nano_cpu_card/de0nano_cpu_card.kicad_pcb (KiCad board)
At the start: 2 copper layers, 160 x 100 mm, 92 parts, among them J1 DIN41617_31P, J2 EXP_HEADER_2x11, J3 GPIO_0_JP1, J4 GPIO_1_JP2, J5 DB9_RS232, P1 DE0Nano_5V_feed, SW1 Rocker_run/halt, SW2 Rocker_dog_off, SW3 Rocker_LC_off, SW4 Button_step, SW5 Button_reset, SW6 Button_qef4, U1 SN74LVC8T245, U2 SN74LVC8T245, U3 SN74LVC8T245, U4 SN74LVC8T245, U5 SN74LVC8T245, U6 SN74LVC8T245, U7 MAX3232EIDR, U8 SN74LVC8T245, U9 SN74LVC8T245

Commit message: Fix R27/R24 schematic-PCB reference mismatch; expand BOM ranges
Root cause of the BOM/CPL mismatch JLCPCB reported: a PCB footprint at
(227.33, 127.49) was still labeled "R27" (value 10k, pad1 on +5V -- a
pull-up resistor) while the schematic calls the same part "R24". A full
schematic-vs-PCB reference diff confirmed this was the only mismatch
(likely a leftover from a schematic rename during the user's own
optimization pass that never got pushed to the PCB via "Update PCB from
Schematic"). Renamed the PCB footprint's Reference property to match the
schematic. pcb drc: still 0 violations, 0 unconnected.

Also regenerated bom.csv/bom_smd_assembly.csv with
--ref-range-delimiter "" so designator lists are plain comma-separated
(e.g. "R1,R2,R3,...") instead of dash-compressed ranges
("R1-R24,R_SW1-R_SW6") -- JLCPCB's BOM parser can't expand ranges,
especially mixed-prefix ones, which was likely contributing to the
mismatch too.

Verified: BOM SMD designator set now matches cpl_smd.csv exactly (72/72,
zero diff either direction).

Co-Authored-By: Claude Sonnet 5 <noreply@anthropic.com>
Parts:
- renumbered R27 to R24
Changed lines of the file:
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@@
 		(descr "Resistor SMD 0603 (1608 Metric), square (rectangular) end terminal, IPC-7351 nominal, (Body size source: IPC-SM-782 page 72, https://www.pcb-3d.com/wordpress/wp-content/uploads/ipc-sm-782a_amendment_1_and_2.pdf)")
 		(tags "resistor")
-		(property "Reference" "R27"
+		(property "Reference" "R24"
 			(at -2.84 -0.09 90)
 			(layer "F.SilkS")
